Commit message: Updated camera_calibration demo - WIP

File: urdf/talos_calibration_camera.urdf (robot description, URDF)
Before this commit: robot talos, 63 links, 62 joints
Joints:
- joint calib_mire_joint: origin xyz=-0.0401 -0.13 -0.35 rpy=-0.60 -2.88 -0.82 -> xyz=-0.08 0.04 -0.52 rpy=1.07 -1.48 -2.57
