Commit message: [tiago/insert_drill] Update airplane skin model

File: urdf/aircraft_skin_with_marker.urdf (robot description, URDF)
Before this commit: robot aircraft_skin, 3 links, 2 joints
Links:
- removed link tag36_11_00020
- added link skin_link; collision mesh filename=package://gerard_bauzil/meshes/AircraftSkinWithFrame.stl; visual mesh filename=package://gerard_bauzil/meshes/AircraftSkinWithFrame.stl
- added link tag36_11_00233; visual mesh filename=package://gerard_bauzil/meshes/apriltag_36h11/tag36_11_0023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 scale=0.0573 0.0573 1.
- link base_link: geometry 
Joints:
- added joint to_skin: type fixed, parent base_link, child skin_link, origin xyz=0 0 -0.09
- joint to_hole: parent base_link -> skin_link
- joint to_tag: child tag36_11_00020 -> tag36_11_00233

Commit message: [URDF] Aircraft skin model comes from rob4fam-models

File: urdf/aircraft_skin_with_marker.urdf (robot description, URDF)
Before this commit: robot aircraft_skin, 4 links, 3 joints
Links:
- link tag36_11_00233: geometry visual mesh filename=package://rob4fam-models/meshes/apriltag_36h11/tag36_11_002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 scale=0.0573 0.0573 1.

Commit message: Changes of skin and tag size

File: urdf/aircraft_skin_with_marker.urdf (robot description, URDF)
Before this commit: robot aircraft_skin, 4 links, 3 joints
Links:
- link skin_link: geometry collision mesh filename=package://rob4fam-models/meshes/AircraftSkinWithFrame.stl; visual mesh filename=package://rob4fam-models/meshes/AircraftSkinWithFrame.stl
- link tag36_11_00233: geometry visual mesh filename=package://gerard_bauzil/meshes/apriltag_36h11/tag36_11_0023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 scale=0.0573 0.0573 1.

Commit message: Fix position of tag on airplane skin.

File: urdf/aircraft_skin_with_marker.urdf (robot description, URDF)
Before this commit: robot aircraft_skin, 4 links, 3 joints
Joints:
- joint to_hole: origin xyz=0.30576 -0.0138 1.5835 rpy=1.8 0 0 -> xyz=0.30576 -0.0138 1.5535 rpy=1.8 0 0
