Commit message: [tiago/deburring] Update cylinder

File: urdf/cylinder.urdf (robot description, URDF)
Before this commit: robot cup, 1 links, 0 joints
Links:
- added link cylinder, mass 1.2; collision mesh filename=package://agimus_demos/meshes/cylinder.stl; visual mesh filename=package://agimus_demos/meshes/cylinder.stl
- added link tag36_11_00100; visual mesh filename=package://gerard_bauzil/meshes/apriltag_36h11/tag36_11_0010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 scale=0.0573 0.0573 1.
- added link tag36_11_00101; visual mesh filename=package://gerard_bauzil/meshes/apriltag_36h11/tag36_11_0010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 scale=0.0573 0.0573 1.
- added link tag36_11_00102; visual mesh filename=package://gerard_bauzil/meshes/apriltag_36h11/tag36_11_0010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 scale=0.0573 0.0573 1.
- added link tag36_11_00103; visual mesh filename=package://gerard_bauzil/meshes/apriltag_36h11/tag36_11_0010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 scale=0.0573 0.0573 1.
- link base_link: mass 1.2 -> None; geometry 
Joints:
- added joint cylinder_fixed_joint: type fixed, parent base_link, child cylinder, origin xyz=0 0 0.5
- added joint to_tag100: type fixed, parent cylinder, child tag36_11_00100, origin xyz=0.5 0 0 rpy=0 1.5707963267948966 0
- added joint to_tag101: type fixed, parent cylinder, child tag36_11_00101, origin xyz=-0.5 0 0 rpy=0 -1.5707963267948966 0
- added joint to_tag102: type fixed, parent cylinder, child tag36_11_00102, origin xyz=0 0.5 0 rpy=-1.5707963267948966 0 0
- added joint to_tag103: type fixed, parent cylinder, child tag36_11_00103, origin xyz=0 -0.5 0 rpy=1.5707963267948966 0 0
