Commit message: [tiago/deburring] Fix models.

File: urdf/P72.urdf (robot description, URDF)
Before this commit: robot p72, 28 links, 27 joints
Links:
- removed link tag36_11_00001_est
- removed link tag36_11_00006_est
- removed link tag36_11_00015_est
- removed link tag36_11_00100_est
- removed link tag36_11_00101_est
- added link tag36_11_00001; visual mesh filename=package://gerard_bauzil/meshes/apriltag_36h11/tag36_11_0000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 scale=0.0495 0.0495 1.
- added link tag36_11_00006; visual mesh filename=package://gerard_bauzil/meshes/apriltag_36h11/tag36_11_0000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 scale=0.1615 0.1615 1.
- added link tag36_11_00015; visual mesh filename=package://gerard_bauzil/meshes/apriltag_36h11/tag36_11_0001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 scale=0.1615 0.1615 1.
- added link tag36_11_00100; visual mesh filename=package://gerard_bauzil/meshes/apriltag_36h11/tag36_11_0010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 scale=0.041 0.041 1.
- added link tag36_11_00101; visual mesh filename=package://gerard_bauzil/meshes/apriltag_36h11/tag36_11_0010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 scale=0.041 0.041 1.
- link base_link: geometry collision box size=0.6 0.1 0.1; collision mesh filename=package://rob4fam-models/meshes/P72.stl scale=0.01 0.01 0.01
Joints:
- removed joint to_tag_00001_est
- removed joint to_tag_00006_est
- removed joint to_tag_00015_est
- removed joint to_tag_00100_est
- removed joint to_tag_00101_est
- added joint to_tag_00001: type fixed, parent base_link, child tag36_11_00001, origin xyz=0.241666609451 -0.0260429212234 0.588386866336 rpy=1.6403222463 -0.0364997670221 0.000742712642255
- added joint to_tag_00006: type fixed, parent base_link, child tag36_11_00006, origin xyz=0.270320819622 -0.00724268033619 0.235261842895 rpy=-3.10995636712 -1.47719252195 -1.60052477825
- added joint to_tag_00015: type fixed, parent base_link, child tag36_11_00015, origin xyz=-0.156366112148 -0.0276786399491 0.490958637679 rpy=1.65921132641 -0.0386653839413 -0.0285749262783
- added joint to_tag_00100: type fixed, parent base_link, child tag36_11_00100, origin xyz=0.0197930637537 -0.0353870621892 0.437950207217 rpy=1.65673314802 -0.0180374390265 -8.37022785993e-05
- added joint to_tag_00101: type fixed, parent base_link, child tag36_11_00101, origin xyz=0.0202331246739 -0.0486944027218 0.701821859147 rpy=1.60759573946 -0.0201753959062 -0.000665864566836
