Commit message: done positioning tag supports and tags

File: urdf/driller_with_qr_drill.urdf (robot description, URDF)
Before this commit: robot driller, 5 links, 4 joints
Links:
- removed link tag_support_link
- added link tag36_11_00023; visual mesh filename=package://gerard_bauzil/meshes/apriltag_36h11/tag36_11_0002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 scale=0.04 0.04 1.
- added link tag_support_link_back, mass 0.001; collision mesh filename=package://gerard_bauzil/meshes/driller/qr_drill_back.stl; visual mesh filename=package://gerard_bauzil/meshes/driller/qr_drill_back.stl
- added link tag_support_link_top, mass 0.001; collision mesh filename=package://gerard_bauzil/meshes/driller/qr_drill_top.stl; visual mesh filename=package://gerard_bauzil/meshes/driller/qr_drill_top.stl
- link base_link: geometry collision mesh filename=package://gerard_bauzil/meshes/driller/BD_drill_2.stl; visual mesh filename=package://gerard_bauzil/meshes/driller/BD_drill_2.stl
- link tag36_11_00230: geometry visual mesh filename=package://gerard_bauzil/meshes/apriltag_36h11/tag36_11_0023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 scale=0.04 0.04 1.
Joints:
- added joint tag_joint_back: type fixed, parent tag_support_link_back, child tag36_11_00230, origin xyz=0 0 0.002
- added joint tag_support_joint_back: type fixed, parent drill_link, child tag_support_link_back, origin xyz=-0.0 0.00 -0.194 rpy=3.141592653589793 0 -1.57079632679
- joint tag_joint: child tag36_11_00230 -> tag36_11_00023; origin xyz=0 0 0.0022 -> xyz=0 0 0.002; parent tag_support_link -> tag_support_link_top
- joint tag_support_joint: child tag_support_link -> tag_support_link_top; origin xyz=0 0.049 0.041 rpy=0 3.141592653589793 0 -> xyz=-0.06 0.00 -0.105 rpy=3.141592653589793 0 -1.57079632679
