Commit message: [ur10/pointing] Add P72 part.

File: urdf/ur10_robot.urdf.xacro (robot description, xacro)
@@ -37,5 +37,5 @@
     <parent link="world" />
     <child link = "support_link" />
-    <origin xyz="0.0 0.0 0.0" rpy="0.0 0.0 ${.5 * M_PI}" />
+    <origin xyz="0.0 0.0 0.0" rpy="0.0 0.0 0.0" />
   </joint>
   <!-- arm -->

Commit message: [ur10/pointing] Switch to robot UR10e.

File: urdf/ur10_robot.urdf.xacro (robot description, xacro)
@@ -1,81 +1,118 @@
 <?xml version="1.0"?>
 <robot xmlns:xacro="http://wiki.ros.org/xacro"
-       name="ur10" >
-  <!-- define global properties -->
-  <xacro:property name="M_PI" value="3.1415926535897931" />
-  <xacro:property name="camera_position_x" value="0.0908" />
-  <xacro:property name="camera_position_y" value="0.08" />
-  <xacro:property name="camera_position_z" value="0.0" />
-  <xacro:property name="camera_orientation_r" value="${.5 * M_PI}" />
-  <xacro:property name="camera_orientation_p" value="0.0" />
-  <xacro:property name="camera_orientation_y" value="0.0" />
+       name="ur10e" >
   <xacro:arg name="transmission_hw_interface" default="hardware_interface/PositionJointInterface"/>
   <!-- common stuff -->
   <xacro:include filename="$(find agimus_demos)/urdf/ur10_gazebo.xacro" />
   <!-- ur10 -->
-  <xacro:include filename="$(find ur_description)/urdf/ur10.urdf.xacro" />
-  <link name="support_link">
-    <inertial>
-      <mass value="200"/>
-      <origin xyz="0 0 0.45"/>
-      <inertia ixx="50"  ixy="0"  ixz="0" iyy="50" iyz="0" izz="50" />
-    </inertial>
-    <visual>
-      <origin xyz="0 0 0.45"/>
-      <geometry>
-	<box size="0.75 0.75 0.9"/>
-      </geometry>
-    </visual>
-    <collision>
-      <origin xyz="0 0 0.45"/>
-      <geometry>
-	<box size="0.75 0.75 0.9"/>
-      </geometry>
-    </collision>
-  </link>
-  <joint name="support_joint" type="fixed">
-    <parent link="world" />
-    <child link = "support_link" />
-    <origin xyz="0.0 0.0 0.0" rpy="0.0 0.0 0.0" />
-  </joint>
-  <!-- arm -->
-  <xacro:ur10_robot prefix="" joint_limited="false"
-    transmission_hw_interface="$(arg transmission_hw_interface)"
-    />
-  <!-- RGB-D sensor -->
-  <xacro:include filename="$(find tiago_description)/urdf/sensors/orbbec_astra.urdf.xacro" />
-  <link name="world" />
-  <joint name="robot_joint" type="fixed">
-    <parent link="support_link" />
-    <child link = "base_link" />
-    <origin xyz="0.0 0.0 0.90" rpy="0.0 0.0 0.0" />
-  </joint>
-  <link name="tool_link">
-    <!--collision>
-      <geometry>
-        <box size="0.02 0.05 0.2"/>
-      </geometry>
-      <origin rpy="0 0 0" xyz="-0.01 0 0"/>
-    </collision>
-    <visual>
-      <geometry>
-        <box size="0.02 0.05 0.2"/>
-      </geometry>
-      <origin rpy="0 0 0" xyz="-0.01 0 0"/>
-    </visual-->
-  </link>
-  <!--xacro:openni_camera_gazebo_v0 name="xtion" /-->
-  <xacro:orbbec_astra name="xtion" parent="tool"
-		      camera_model="orbbec-astra'"
-		      extrinsic_calibration_dir="$(find tiago_description_calibration)/urdf/calibration">
-    <origin xyz="${camera_position_x} ${camera_position_y} ${camera_position_z}"
-	    rpy="${camera_orientation_r} ${camera_orientation_p}
-		 ${camera_orientation_y}" />
-    <optical_origin xyz="0 0 0" rpy="${-0.5 * M_PI} 0 ${-.5 * M_PI}"/>
-  </xacro:orbbec_astra>
-  <joint name="tool_joint" type="fixed">
-    <parent link="ee_link"/>
-    <child link="tool_link" />
-    <origin xyz="0.0 0.0 0.0" rpy="0.0 0.0 0.0" />
-  </joint>
+  <xacro:include filename="$(find ur_description)/urdf/ur10e.xacro" />
+    <!-- <xacro:include filename="$(find ur_description)/urdf/ur10.urdf.xacro" /> -->
+   <link name="world" />
+    <!-- define global properties -->
+    <xacro:property name="M_PI" value="3.1415926535897931" />
+    <xacro:property name="camera_position_x" value="0.0908" />
+    <xacro:property name="camera_position_y" value="0.08" />
+    <xacro:property name="camera_position_z" value="0.0" />
+    <xacro:property name="camera_orientation_r" value="${.5 * M_PI}" />
+    <xacro:property name="camera_orientation_p" value="0.0" />
+    <xacro:property name="camera_orientation_y" value="0.0" />
+    <link name="support_link">
+      <inertial>
+        <mass value="200"/>
+        <origin xyz="0 0 0.45"/>
+        <inertia ixx="50"  ixy="0"  ixz="0" iyy="50" iyz="0" izz="50" />
+      </inertial>
+      <visual>
+        <origin xyz="0 0 0.45"/>
+        <geometry>
+    <box size="0.75 0.75 0.9"/>
+        </geometry>
+      </visual>
+      <collision>
+        <origin xyz="0 0 0.45"/>
+        <geometry>
+    <box size="0.75 0.75 0.9"/>
+        </geometry>
+      </collision>
+    </link>
+    <joint name="support_joint" type="fixed">
+      <parent link="world" />
+      <child link = "support_link" />
+      <origin xyz="0.0 0.0 0.0" rpy="0.0 0.0 0.0" />
+    </joint>
+    <xacro:include filename="$(find tiago_description)/urdf/sensors/orbbec_astra.urdf.xacro" />
+    <!-- <link name="world" /> -->
+    <joint name="robot_joint" type="fixed">
+      <parent link="support_link" />
+      <child link = "base_link" />
+      <origin xyz="0.2 0.0 0.90" rpy="0.0 0.0 -1.5707963" />
+    </joint>
+    <link name="tool_link">
+      <!--collision>
+        <geometry>
+          <box size="0.02 0.05 0.2"/>
+        </geometry>
+        <origin rpy="0 0 0" xyz="-0.01 0 0"/>
+      </collision>
+      <visual>
+        <geometry>
+          <box size="0.02 0.05 0.2"/>
+        </geometry>
+        <origin rpy="0 0 0" xyz="-0.01 0 0"/>
+      </visual-->
+    </link>
+  <link name="collision_cylinder">
+   <visual>
+     <origin xyz="0 0 0" rpy="0 0 0" />
+     <geometry>
+       <cylinder radius="0.045" length="0.115"/>
+     </geometry>
+     <material name="black">
+       <color rgba="0 0 0 1"/>
+     </material>
+   </visual>
+   <collision>
+     <origin xyz="0 0 0" rpy="0 0 0"/>
+     <geometry>
+       <cylinder radius="0.045" length="0.115"/>
+     </geometry>
+   </collision>
+ </link>
+ <joint name="collision_cylinder_joint" type="fixed">
+    <parent link="wrist_3_link" />
+    <child link = "collision_cylinder" />
+    <origin xyz="0.0 0.0 0.05" rpy="0.0 0.0 ${pi/2.0}" />
+ </joint>
+    <joint name="ee_fixed_joint" type="fixed">
+     <parent link="wrist_3_link" />
+     <child link = "ee_link" />
+     <origin xyz="0.0 0.0 0.117" rpy="0.0 0.0 ${pi/2.0}" />
+   </joint>
+   <link name="ee_link">
+     <collision>
+       <geometry>
+         <box size="0.01 0.01 0.01"/>
+       </geometry>
+       <origin rpy="0 0 0" xyz="-0.01 0 0"/>
+     </collision>
+     <visual>
+       <geometry>
+         <box size="0.01 0.01 0.01"/>
+       </geometry>
+       <origin rpy="0 0 0" xyz="-0.01 0 0"/>
+     </visual>
+   </link>
+   <xacro:orbbec_astra name="xtion" parent="tool"
+           camera_model="orbbec-astra'"
+           extrinsic_calibration_dir="$(find tiago_description_calibration)/urdf/calibration">
+     <origin xyz="${camera_position_x} ${camera_position_y} ${camera_position_z}"
+       rpy="${camera_orientation_r} ${camera_orientation_p}
+      ${camera_orientation_y}" />
+     <optical_origin xyz="0 0 0" rpy="${-0.5 * M_PI} 0 ${-.5 * M_PI}"/>
+   </xacro:orbbec_astra>
+   <joint name="tool_joint" type="fixed">
+     <parent link="ee_link"/>
+     <child link="tool_link" />
+     <origin xyz="0.0 0.0 0.0" rpy="0.0 0.0 0.0" />
+   </joint>
 </robot>

Commit message: [ur10/pointing] Update script and model of robot support.

File: urdf/ur10_robot.urdf.xacro (robot description, xacro)
@@ -24,13 +24,13 @@
       </inertial>
       <visual>
-        <origin xyz="0 0 0.45"/>
+        <origin xyz="-0.4 0 0.45"/>
         <geometry>
-    <box size="0.75 0.75 0.9"/>
+	  <box size="1.0 1.2 0.9"/>
         </geometry>
       </visual>
       <collision>
-        <origin xyz="0 0 0.45"/>
+        <origin xyz="-0.4 0 0.45"/>
         <geometry>
-    <box size="0.75 0.75 0.9"/>
+	  <box size="1.0 1.2 0.9"/>
         </geometry>
       </collision>
@@ -46,5 +46,5 @@
       <parent link="support_link" />
       <child link = "base_link" />
-      <origin xyz="0.2 0.0 0.90" rpy="0.0 0.0 -1.5707963" />
+      <origin xyz="0.0 0.0 0.90" rpy="0.0 0.0 -1.5707963" />
     </joint>
     <link name="tool_link">
