Commit message: [tiago/deburring] Update HPP related files.

File: urdf/P72-with-table.urdf (robot description, URDF)
Before this commit: robot p72, 21 links, 20 joints
Links:
- added link table_link, mass 2.2; collision box size=.02 .02 .72; collision box size=.02 .02 .72
Joints:
- added joint to_table: type fixed, parent base_link, child table_link, origin xyz=0.0 0.35 -0.8

Commit message: [tiago/deburring] Update models.

File: urdf/P72-with-table.urdf (robot description, URDF)
Before this commit: robot p72, 22 links, 21 joints
Links:
- added link tag36_11_00001; visual mesh filename=package://gerard_bauzil/meshes/apriltag_36h11/tag36_11_0000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 scale=0.0495 0.0495 1.
- added link tag36_11_00006; visual mesh filename=package://gerard_bauzil/meshes/apriltag_36h11/tag36_11_0000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 scale=0.1615 0.1615 1.
- added link tag36_11_00015; visual mesh filename=package://gerard_bauzil/meshes/apriltag_36h11/tag36_11_0001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 scale=0.1615 0.1615 1.
- added link tag36_11_00100_cao; visual mesh filename=package://gerard_bauzil/meshes/apriltag_36h11/tag36_11_0010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 scale=0.041 0.041 1.
- added link tag36_11_00101_cao; visual mesh filename=package://gerard_bauzil/meshes/apriltag_36h11/tag36_11_0010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 scale=0.041 0.041 1.
- added link tag_100_base_link
- added link tag_101_base_link
- link base_link: geometry collision box size=0.6 0.1 0.1; collision mesh filename=package://rob4fam-models/meshes/P72.stl scale=0.01 0.01 0.01
- link tag36_11_00100: geometry visual mesh filename=package://gerard_bauzil/meshes/apriltag_36h11/tag36_11_0010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 scale=0.041 0.041 1.
- link tag36_11_00101: geometry visual mesh filename=package://gerard_bauzil/meshes/apriltag_36h11/tag36_11_0010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 scale=0.041 0.041 1.
Joints:
- removed joint to_tag_100
- removed joint to_tag_101
- added joint to_tag_00001: type fixed, parent base_link, child tag36_11_00001, origin xyz=0.241666609451 -0.0260429212234 0.588386866336 rpy=1.6403222463 -0.0364997670221 0.000742712642255
- added joint to_tag_00006: type fixed, parent base_link, child tag36_11_00006, origin xyz=0.270320819622 -0.00724268033619 0.235261842895 rpy=-3.10995636712 -1.47719252195 -1.60052477825
- added joint to_tag_00015: type fixed, parent base_link, child tag36_11_00015, origin xyz=-0.156366112148 -0.0276786399491 0.490958637679 rpy=1.65921132641 -0.0386653839413 -0.0285749262783
- added joint to_tag_00100: type fixed, parent base_link, child tag36_11_00100, origin xyz=0.0197930637537 -0.0353870621892 0.437950207217 rpy=1.65673314802 -0.0180374390265 -8.37022785993e-05
- added joint to_tag_00101: type fixed, parent base_link, child tag36_11_00101, origin xyz=0.0202331246739 -0.0486944027218 0.701821859147 rpy=1.60759573946 -0.0201753959062 -0.000665864566836
- added joint to_tag_100_base: type fixed, parent base_link, child tag_100_base_link, origin xyz=0.02 -0.031 0.44 rpy=1.6 0 0
- added joint to_tag_100_cao: type fixed, parent tag_100_base_link, child tag36_11_00100_cao, origin xyz=0. 0. 0.004 rpy=0 0 0
- added joint to_tag_101_base: type fixed, parent base_link, child tag_101_base_link, origin xyz=0.02 -0.045 0.70 rpy=1.6 0 0
- added joint to_tag_101_cao: type fixed, parent tag_101_base_link, child tag36_11_00101_cao, origin xyz=0. 0. 0.004 rpy=0 0 0
- joint to_hole_01: parent tag36_11_00100 -> tag_100_base_link
- joint to_hole_02: parent tag36_11_00100 -> tag_100_base_link
- joint to_hole_03: parent tag36_11_00100 -> tag_100_base_link
- joint to_hole_04: parent tag36_11_00100 -> tag_100_base_link
- joint to_hole_05: parent tag36_11_00100 -> tag_100_base_link
- joint to_hole_06: parent tag36_11_00100 -> tag_100_base_link
- joint to_hole_07: parent tag36_11_00100 -> tag_100_base_link
- joint to_hole_08: parent tag36_11_00100 -> tag_100_base_link
- joint to_hole_09: parent tag36_11_00100 -> tag_100_base_link
- joint to_hole_10: parent tag36_11_00100 -> tag_100_base_link
- joint to_hole_11: parent tag36_11_00100 -> tag_100_base_link
- joint to_hole_12: parent tag36_11_00100 -> tag_100_base_link
- joint to_hole_13: parent tag36_11_00101 -> tag_101_base_link
- joint to_hole_14: parent tag36_11_00101 -> tag_101_base_link
- joint to_hole_15: parent tag36_11_00101 -> tag_101_base_link
- joint to_hole_16: parent tag36_11_00101 -> tag_101_base_link
- joint to_hole_17: parent tag36_11_00101 -> tag_101_base_link
- joint to_hole_18: parent tag36_11_00101 -> tag_101_base_link

File: urdf/P72.urdf (robot description, URDF)
Before this commit: robot p72, 21 links, 20 joints
Links:
- removed link tag36_11_00100
- removed link tag36_11_00101
- added link tag36_11_00001_est; visual mesh filename=package://gerard_bauzil/meshes/apriltag_36h11/tag36_11_0000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 scale=0.0495 0.0495 1.
- added link tag36_11_00006_est; visual mesh filename=package://gerard_bauzil/meshes/apriltag_36h11/tag36_11_0000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 scale=0.1615 0.1615 1.
- added link tag36_11_00015_est; visual mesh filename=package://gerard_bauzil/meshes/apriltag_36h11/tag36_11_0001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 scale=0.1615 0.1615 1.
- added link tag36_11_00100_cao; visual mesh filename=package://gerard_bauzil/meshes/apriltag_36h11/tag36_11_0010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 scale=0.041 0.041 1.
- added link tag36_11_00100_est; visual mesh filename=package://gerard_bauzil/meshes/apriltag_36h11/tag36_11_0010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 scale=0.041 0.041 1.
- added link tag36_11_00101_cao; visual mesh filename=package://gerard_bauzil/meshes/apriltag_36h11/tag36_11_0010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 scale=0.041 0.041 1.
- added link tag36_11_00101_est; visual mesh filename=package://gerard_bauzil/meshes/apriltag_36h11/tag36_11_0010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 scale=0.041 0.041 1.
- added link tag_100_base_link
- added link tag_101_base_link
Joints:
- removed joint to_tag_100
- removed joint to_tag_101
- added joint to_tag_00001_est: type fixed, parent base_link, child tag36_11_00001_est, origin xyz=0.241666609451 -0.0260429212234 0.588386866336 rpy=1.6403222463 -0.0364997670221 0.000742712642255
- added joint to_tag_00006_est: type fixed, parent base_link, child tag36_11_00006_est, origin xyz=0.270320819622 -0.00724268033619 0.235261842895 rpy=-3.10995636712 -1.47719252195 -1.60052477825
- added joint to_tag_00015_est: type fixed, parent base_link, child tag36_11_00015_est, origin xyz=-0.156366112148 -0.0276786399491 0.490958637679 rpy=1.65921132641 -0.0386653839413 -0.0285749262783
- added joint to_tag_00100_est: type fixed, parent base_link, child tag36_11_00100_est, origin xyz=0.0197930637537 -0.0353870621892 0.437950207217 rpy=1.65673314802 -0.0180374390265 -8.37022785993e-05
- added joint to_tag_00101_est: type fixed, parent base_link, child tag36_11_00101_est, origin xyz=0.0202331246739 -0.0486944027218 0.701821859147 rpy=1.60759573946 -0.0201753959062 -0.000665864566836
- added joint to_tag_100_base: type fixed, parent base_link, child tag_100_base_link, origin xyz=0.02 -0.031 0.44 rpy=1.6 0 0
- added joint to_tag_100_cao: type fixed, parent tag_100_base_link, child tag36_11_00100_cao, origin xyz=0. 0. 0.004 rpy=0 0 0
- added joint to_tag_101_base: type fixed, parent base_link, child tag_101_base_link, origin xyz=0.02 -0.045 0.70 rpy=1.6 0 0
- added joint to_tag_101_cao: type fixed, parent tag_101_base_link, child tag36_11_00101_cao, origin xyz=0. 0. 0.004 rpy=0 0 0
- joint to_hole_01: parent tag36_11_00100 -> tag_100_base_link
- joint to_hole_02: parent tag36_11_00100 -> tag_100_base_link
- joint to_hole_03: parent tag36_11_00100 -> tag_100_base_link
- joint to_hole_04: parent tag36_11_00100 -> tag_100_base_link
- joint to_hole_05: parent tag36_11_00100 -> tag_100_base_link
- joint to_hole_06: parent tag36_11_00100 -> tag_100_base_link
- joint to_hole_07: parent tag36_11_00100 -> tag_100_base_link
- joint to_hole_08: parent tag36_11_00100 -> tag_100_base_link
- joint to_hole_09: parent tag36_11_00100 -> tag_100_base_link
- joint to_hole_10: parent tag36_11_00100 -> tag_100_base_link
- joint to_hole_11: parent tag36_11_00100 -> tag_100_base_link
- joint to_hole_12: parent tag36_11_00100 -> tag_100_base_link
- joint to_hole_13: parent tag36_11_00101 -> tag_101_base_link
- joint to_hole_14: parent tag36_11_00101 -> tag_101_base_link
- joint to_hole_15: parent tag36_11_00101 -> tag_101_base_link
- joint to_hole_16: parent tag36_11_00101 -> tag_101_base_link
- joint to_hole_17: parent tag36_11_00101 -> tag_101_base_link
- joint to_hole_18: parent tag36_11_00101 -> tag_101_base_link

Commit message: [tiago/deburring] Update part model + scripts

File: urdf/P72-with-table.urdf (robot description, URDF)
Before this commit: robot p72, 29 links, 28 joints
Links:
- removed link tag36_11_00100_cao
- removed link tag36_11_00101_cao
- removed link tag_100_base_link
- removed link tag_101_base_link
- link hole_01_link: geometry visual sphere radius=0.005
- link hole_02_link: geometry visual sphere radius=0.005
- link hole_03_link: geometry visual sphere radius=0.005
- link hole_04_link: geometry visual sphere radius=0.005
- link hole_05_link: geometry visual sphere radius=0.005
- link hole_06_link: geometry visual sphere radius=0.005
- link hole_07_link: geometry visual sphere radius=0.005
- link hole_08_link: geometry visual sphere radius=0.005
- link hole_09_link: geometry visual sphere radius=0.005
- link hole_10_link: geometry visual sphere radius=0.005
- link hole_11_link: geometry visual sphere radius=0.005
- link hole_12_link: geometry visual sphere radius=0.005
- link hole_13_link: geometry visual sphere radius=0.005
- link hole_14_link: geometry visual sphere radius=0.005
- link hole_15_link: geometry visual sphere radius=0.005
- link hole_16_link: geometry visual sphere radius=0.005
- link hole_17_link: geometry visual sphere radius=0.005
- link hole_18_link: geometry visual sphere radius=0.005
- link tag36_11_00001: geometry visual mesh filename=package://gerard_bauzil/meshes/apriltag_36h11/tag36_11_0000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 scale=0.0845 0.0845 1.
- link tag36_11_00015: geometry visual mesh filename=package://gerard_bauzil/meshes/apriltag_36h11/tag36_11_0001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 scale=0.0845 0.0845 1.
Joints:
- removed joint to_tag_100_base
- removed joint to_tag_100_cao
- removed joint to_tag_101_base
- removed joint to_tag_101_cao
- joint to_hole_01: origin xyz=-0.045 -0.003 0.0 rpy=0 0 0 -> xyz=-0.0231859078401 -0.0282814474512 0.441118345594 rpy=-0.06403080615 0.0647848229269 -1.55908144855; parent tag_100_base_link -> base_link
- joint to_hole_02: origin xyz=-0.023 0.033 0.0 rpy=0 0 0 -> xyz=-0.000463757557886 -0.0305306738819 0.471682850952 rpy=-0.06403080615 0.0647848229269 -1.55908144855; parent tag_100_base_link -> base_link
- joint to_hole_03: origin xyz=0.022 0.033 0.0 rpy=0 0 0 -> xyz=0.0461839113985 -0.0310339220481 0.471016257947 rpy=-0.06403080615 0.0647848229269 -1.55908144855; parent tag_100_base_link -> base_link
- joint to_hole_04: origin xyz=0.037 -0.003 0.0 rpy=0 0 0 -> xyz=0.0685148465977 -0.0290956950629 0.437109953868 rpy=-0.06403080615 0.0647848229269 -1.55908144855; parent tag_100_base_link -> base_link
- joint to_hole_05: origin xyz=0.022 -0.035 0.0 rpy=0 0 0 -> xyz=0.0445673657398 -0.0269147516117 0.407819156194 rpy=-0.06403080615 0.0647848229269 -1.55908144855; parent tag_100_base_link -> base_link
- joint to_hole_06: origin xyz=-0.023 -0.035 0.0 rpy=0 0 0 -> xyz=-0.000455903779824 -0.0264076500538 0.408133038324 rpy=-0.06403080615 0.0647848229269 -1.55908144855; parent tag_100_base_link -> base_link
- joint to_hole_07: origin xyz=-0.045 -0.07 0.0 rpy=0 0 0 -> xyz=-0.0208802619903 -0.0238630597283 0.37260115984 rpy=-0.06403080615 0.0647848229269 -1.55908144855; parent tag_100_base_link -> base_link
- joint to_hole_08: origin xyz=-0.023 -0.11 0.0 rpy=0 0 0 -> xyz=-0.00240257087843 -0.0215015648055 0.332866785156 rpy=-0.06403080615 0.0647848229269 -1.55908144855; parent tag_100_base_link -> base_link
- joint to_hole_09: origin xyz=0.022 -0.11 0.0 rpy=0 0 0 -> xyz=0.0441438434551 -0.0220229148067 0.332497480315 rpy=-0.06403080615 0.0647848229269 -1.55908144855; parent tag_100_base_link -> base_link
- joint to_hole_10: origin xyz=0.037 -0.07 0.0 rpy=0 0 0 -> xyz=0.0643483206286 -0.0247997737006 0.37164903109 rpy=-0.06403080615 0.0647848229269 -1.55908144855; parent tag_100_base_link -> base_link
- joint to_hole_11: origin xyz=-0.035 0.095 0.005 rpy=0 0 0 -> xyz=-0.0183193680998 -0.0342875833339 0.532812497719 rpy=-0.06403080615 0.0647848229269 -1.55908144855; parent tag_100_base_link -> base_link
- joint to_hole_12: origin xyz=0.05 0.095 0.005 rpy=0 0 0 -> xyz=0.0691214440517 -0.035208122937 0.53121160951 rpy=-0.06403080615 0.0647848229269 -1.55908144855; parent tag_100_base_link -> base_link
- joint to_hole_13: origin xyz=-0.04 -0.105 0.0 rpy=0 0 0 -> xyz=-0.0173508237974 -0.0384699820474 0.597101150222 rpy=-0.06403080615 0.0647848229269 -1.55908144855; parent tag_101_base_link -> base_link
- joint to_hole_14: origin xyz=-0.04 -0.055 0.0 rpy=0 0 0 -> xyz=-0.0165201674869 -0.0417052933682 0.646817190801 rpy=-0.06403080615 0.0647848229269 -1.55908144855; parent tag_101_base_link -> base_link
- joint to_hole_15: origin xyz=-0.04 -0.01 0.0 rpy=0 0 0 -> xyz=-0.0157844883883 -0.0445989234655 0.691284029836 rpy=-0.06403080615 0.0647848229269 -1.55908144855; parent tag_101_base_link -> base_link
- joint to_hole_16: origin xyz=0.05 -0.01 0.0 rpy=0 0 0 -> xyz=0.0717634019701 -0.0454885386124 0.689187166127 rpy=-0.06403080615 0.0647848229269 -1.55908144855; parent tag_101_base_link -> base_link
- joint to_hole_17: origin xyz=0.05 -0.055 0.0 rpy=0 0 0 -> xyz=0.0710534490762 -0.0426129907748 0.644994384573 rpy=-0.06403080615 0.0647848229269 -1.55908144855; parent tag_101_base_link -> base_link
- joint to_hole_18: origin xyz=0.05 -0.105 0.0 rpy=0 0 0 -> xyz=0.0699350800666 -0.039412993952 0.595874600682 rpy=-0.06403080615 0.0647848229269 -1.55908144855; parent tag_101_base_link -> base_link
- joint to_tag_00001: origin xyz=0.241666609451 -0.0260429212234 0.588386866336 rpy=1.6403222463 -0.0364997670221 0.000742712642255 -> xyz=0.160353229673 -0.0402800139396 0.592911176226 rpy=1.63558131631 -0.00225646482702 -0.0118612667906
- joint to_tag_00006: origin xyz=0.270320819622 -0.00724268033619 0.235261842895 rpy=-3.10995636712 -1.47719252195 -1.60052477825 -> xyz=0.289039801823 -0.0185894364178 0.235356143456 rpy=-2.88571492705 -1.5038280042 -1.83893893187
- joint to_tag_00015: origin xyz=-0.156366112148 -0.0276786399491 0.490958637679 rpy=1.65921132641 -0.0386653839413 -0.0285749262783 -> xyz=-0.132714992453 -0.0338492746834 0.546713277339 rpy=1.63558443485 -0.0100636021863 -0.0123677826844
- joint to_tag_00100: origin xyz=0.0197930637537 -0.0353870621892 0.437950207217 rpy=1.65673314802 -0.0180374390265 -8.37022785993e-05 -> xyz=0.0208917170125 -0.0327790965142 0.440695684094 rpy=1.63559977055 0.0239548219158 -0.0101604937887
- joint to_tag_00101: origin xyz=0.0202331246739 -0.0486944027218 0.701821859147 rpy=1.60759573946 -0.0201753959062 -0.000665864566836 -> xyz=0.0295741667779 -0.0501954344754 0.707566863227 rpy=1.6355812991 -0.00213025081185 -0.0118530770043

Commit message: [tiago/deburring] update model.

File: urdf/P72-with-table.urdf (robot description, URDF)
Before this commit: robot p72, 25 links, 24 joints
Joints:
- joint to_hole_01: origin xyz=-0.0231859078401 -0.0282814474512 0.441118345594 rpy=-0.06403080615 0.0647848229269 -1.55908144855 -> xyz=-0.0231859078401 -0.0282814474512 0.441118345594 rpy=-0.06403080615 -0.0647848229269 1.55908144855
- joint to_hole_02: origin xyz=-0.000463757557886 -0.0305306738819 0.471682850952 rpy=-0.06403080615 0.0647848229269 -1.55908144855 -> xyz=-0.000463757557886 -0.0305306738819 0.471682850952 rpy=-0.06403080615 -0.0647848229269 1.55908144855
- joint to_hole_03: origin xyz=0.0461839113985 -0.0310339220481 0.471016257947 rpy=-0.06403080615 0.0647848229269 -1.55908144855 -> xyz=0.0461839113985 -0.0310339220481 0.471016257947 rpy=-0.06403080615 -0.0647848229269 1.55908144855
- joint to_hole_04: origin xyz=0.0685148465977 -0.0290956950629 0.437109953868 rpy=-0.06403080615 0.0647848229269 -1.55908144855 -> xyz=0.0685148465977 -0.0290956950629 0.437109953868 rpy=-0.06403080615 -0.0647848229269 1.55908144855
- joint to_hole_05: origin xyz=0.0445673657398 -0.0269147516117 0.407819156194 rpy=-0.06403080615 0.0647848229269 -1.55908144855 -> xyz=0.0445673657398 -0.0269147516117 0.407819156194 rpy=-0.06403080615 -0.0647848229269 1.55908144855
- joint to_hole_06: origin xyz=-0.000455903779824 -0.0264076500538 0.408133038324 rpy=-0.06403080615 0.0647848229269 -1.55908144855 -> xyz=-0.000455903779824 -0.0264076500538 0.408133038324 rpy=-0.06403080615 -0.0647848229269 1.55908144855
- joint to_hole_07: origin xyz=-0.0208802619903 -0.0238630597283 0.37260115984 rpy=-0.06403080615 0.0647848229269 -1.55908144855 -> xyz=-0.0208802619903 -0.0238630597283 0.37260115984 rpy=-0.06403080615 -0.0647848229269 1.55908144855
- joint to_hole_08: origin xyz=-0.00240257087843 -0.0215015648055 0.332866785156 rpy=-0.06403080615 0.0647848229269 -1.55908144855 -> xyz=-0.00240257087843 -0.0215015648055 0.332866785156 rpy=-0.06403080615 -0.0647848229269 1.55908144855
- joint to_hole_09: origin xyz=0.0441438434551 -0.0220229148067 0.332497480315 rpy=-0.06403080615 0.0647848229269 -1.55908144855 -> xyz=0.0441438434551 -0.0220229148067 0.332497480315 rpy=-0.06403080615 -0.0647848229269 1.55908144855
- joint to_hole_10: origin xyz=0.0643483206286 -0.0247997737006 0.37164903109 rpy=-0.06403080615 0.0647848229269 -1.55908144855 -> xyz=0.0643483206286 -0.0247997737006 0.37164903109 rpy=-0.06403080615 -0.0647848229269 1.55908144855
- joint to_hole_11: origin xyz=-0.0183193680998 -0.0342875833339 0.532812497719 rpy=-0.06403080615 0.0647848229269 -1.55908144855 -> xyz=-0.0183193680998 -0.0342875833339 0.532812497719 rpy=-0.06403080615 -0.0647848229269 1.55908144855
- joint to_hole_12: origin xyz=0.0691214440517 -0.035208122937 0.53121160951 rpy=-0.06403080615 0.0647848229269 -1.55908144855 -> xyz=0.0691214440517 -0.035208122937 0.53121160951 rpy=-0.06403080615 -0.0647848229269 1.55908144855
- joint to_hole_13: origin xyz=-0.0173508237974 -0.0384699820474 0.597101150222 rpy=-0.06403080615 0.0647848229269 -1.55908144855 -> xyz=-0.0173508237974 -0.0384699820474 0.597101150222 rpy=-0.06403080615 -0.0647848229269 1.55908144855
- joint to_hole_14: origin xyz=-0.0165201674869 -0.0417052933682 0.646817190801 rpy=-0.06403080615 0.0647848229269 -1.55908144855 -> xyz=-0.0165201674869 -0.0417052933682 0.646817190801 rpy=-0.06403080615 -0.0647848229269 1.55908144855
- joint to_hole_15: origin xyz=-0.0157844883883 -0.0445989234655 0.691284029836 rpy=-0.06403080615 0.0647848229269 -1.55908144855 -> xyz=-0.0157844883883 -0.0445989234655 0.691284029836 rpy=-0.06403080615 -0.0647848229269 1.55908144855
- joint to_hole_16: origin xyz=0.0717634019701 -0.0454885386124 0.689187166127 rpy=-0.06403080615 0.0647848229269 -1.55908144855 -> xyz=0.0717634019701 -0.0454885386124 0.689187166127 rpy=-0.06403080615 -0.0647848229269 1.55908144855
- joint to_hole_17: origin xyz=0.0710534490762 -0.0426129907748 0.644994384573 rpy=-0.06403080615 0.0647848229269 -1.55908144855 -> xyz=0.0710534490762 -0.0426129907748 0.644994384573 rpy=-0.06403080615 -0.0647848229269 1.55908144855
- joint to_hole_18: origin xyz=0.0699350800666 -0.039412993952 0.595874600682 rpy=-0.06403080615 0.0647848229269 -1.55908144855 -> xyz=0.0699350800666 -0.039412993952 0.595874600682 rpy=-0.06403080615 -0.0647848229269 1.55908144855

Commit message: [tiago/deburring] Update Python script and models

File: urdf/P72-with-table.urdf (robot description, URDF)
Before this commit: robot p72, 25 links, 24 joints
Links:
- link base_link: geometry collision box size=0.6 0.15 0.15; collision mesh filename=package://rob4fam-models/meshes/P72.stl scale=0.01 0.01 0.01
