Commit message: [tiago/deburring] Add calibrated P72 model

File: urdf/P72-with-table.urdf (robot description, URDF)
Before this commit: robot p72, 25 links, 24 joints
Links:
- added link hole_00_link; visual sphere radius=0.005
- added link hole_19_link; visual sphere radius=0.005
- added link hole_20_link; visual sphere radius=0.005
- added link hole_21_link; visual sphere radius=0.005
- added link hole_22_link; visual sphere radius=0.005
- added link hole_23_link; visual sphere radius=0.005
- added link hole_24_link; visual sphere radius=0.005
- added link hole_25_link; visual sphere radius=0.005
- added link hole_26_link; visual sphere radius=0.005
- added link hole_27_link; visual sphere radius=0.005
- added link hole_28_link; visual sphere radius=0.005
- added link hole_29_link; visual sphere radius=0.005
- added link hole_30_link; visual sphere radius=0.005
- added link hole_31_link; visual sphere radius=0.005
- added link hole_32_link; visual sphere radius=0.005
- added link hole_33_link; visual sphere radius=0.005
- added link hole_34_link; visual sphere radius=0.005
- added link hole_35_link; visual sphere radius=0.005
- added link hole_36_link; visual sphere radius=0.005
- added link hole_37_link; visual sphere radius=0.005
- added link tag36_11_00002; visual mesh filename=package://gerard_bauzil/meshes/apriltag_36h11/tag36_11_0000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 scale=0.053 0.053 1.
- added link tag36_11_00003; visual mesh filename=package://gerard_bauzil/meshes/apriltag_36h11/tag36_11_0000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 scale=0.053 0.053 1.
- added link tag36_11_00004; visual mesh filename=package://gerard_bauzil/meshes/apriltag_36h11/tag36_11_0000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 scale=0.053 0.053 1.
- link tag36_11_00006: geometry visual mesh filename=package://gerard_bauzil/meshes/apriltag_36h11/tag36_11_0000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 scale=0.0845 0.0845 1.
Joints:
- added joint to_hole_00: type fixed, parent base_link, child hole_00_link, origin xyz=-0.166815918156 -0.0427314643607 0.689768700188 rpy=-0.0640321358084 -0.0647859936191 1.55908414531
- added joint to_hole_19: type fixed, parent base_link, child hole_19_link, origin xyz=0.0676823414569 -0.0291717367669 0.438442735487 rpy=-0.0640321358084 -0.0647859936191 1.55908414531
- added joint to_hole_20: type fixed, parent base_link, child hole_20_link, origin xyz=0.0466270535706 -0.0309939122152 0.470328534663 rpy=-0.0640321358084 -0.0647859936191 1.55908414531
- added joint to_hole_21: type fixed, parent base_link, child hole_21_link, origin xyz=-0.0211758097543 -0.0238817962681 0.372951226012 rpy=-0.0640321358084 -0.0647859936191 1.55908414531
- added joint to_hole_22: type fixed, parent base_link, child hole_22_link, origin xyz=-0.00265232492397 -0.0214048675679 0.331430916265 rpy=-0.0640321358084 -0.0647859936191 1.55908414531
- added joint to_hole_23: type fixed, parent base_link, child hole_23_link, origin xyz=0.0445434344292 -0.021991831719 0.331957625953 rpy=-0.0640321358084 -0.0647859936191 1.55908414531
- added joint to_hole_24: type fixed, parent base_link, child hole_24_link, origin xyz=0.0651477595884 -0.0247764180189 0.37115622644 rpy=-0.0640321358084 -0.0647859936191 1.55908414531
- added joint to_hole_25: type fixed, parent base_link, child hole_25_link, origin xyz=-0.064504007426 -0.0159695547558 0.258823459798 rpy=-0.0640321358084 -0.0647859936191 1.55908414531
- added joint to_hole_26: type fixed, parent base_link, child hole_26_link, origin xyz=-0.0984845919704 -0.0121441264254 0.205997349468 rpy=-0.0640321358084 -0.0647859936191 1.55908414531
- added joint to_hole_27: type fixed, parent base_link, child hole_27_link, origin xyz=0.102726204679 -0.0174611899519 0.251624383672 rpy=-0.0640321358084 -0.0647859936191 1.55908414531
- added joint to_hole_28: type fixed, parent base_link, child hole_28_link, origin xyz=0.104743399249 0.0130284323996 0.241182377786 rpy=-1.70979382248 -0.76557361026 -3.04842222337
- added joint to_hole_29: type fixed, parent base_link, child hole_29_link, origin xyz=0.0479809773644 0.278664639966 0.455172061897 rpy=-1.43338884326 0.276368114583 1.58182234414
- added joint to_hole_30: type fixed, parent base_link, child hole_30_link, origin xyz=-0.0114167174748 0.281745848087 0.498838668863 rpy=-1.8917737621 0.250659632952 1.50033157495
- added joint to_hole_31: type fixed, parent base_link, child hole_31_link, origin xyz=-0.0312547275123 0.284154076218 0.539726344304 rpy=-2.21546992664 0.534043741073 1.20554044441
- added joint to_hole_32: type fixed, parent base_link, child hole_32_link, origin xyz=-0.0488979605901 0.287087954303 0.581292765755 rpy=-2.25648458741 0.360820672617 1.29857569528
- added joint to_hole_33: type fixed, parent base_link, child hole_33_link, origin xyz=-0.0645676676101 0.288844357991 0.625612000194 rpy=-3.12218734873 -1.20487785721 3.04938840946
- added joint to_hole_34: type fixed, parent base_link, child hole_34_link, origin xyz=-0.086235960475 0.291866090557 0.665538827329 rpy=3.07565034697 -1.24476911814 3.09128169578
- added joint to_hole_35: type fixed, parent base_link, child hole_35_link, origin xyz=-0.0181148648809 0.292225548538 0.238329406869 rpy=-1.90145827427 -1.49236800609 0.374570802956
- added joint to_hole_36: type fixed, parent base_link, child hole_36_link, origin xyz=-0.0577110509484 0.289545685621 0.180503344604 rpy=-2.31264009349 -1.54712996346 0.765146825955
- added joint to_hole_37: type fixed, parent base_link, child hole_37_link, origin xyz=-0.0652507273193 0.279317534307 0.0871087391981 rpy=2.64379590214 -1.4845807824 2.08337128465
- added joint to_tag_00002: type fixed, parent base_link, child tag36_11_00002, origin xyz=0.0252040551767 0.290936526509 0.367238386507 rpy=1.54992774545 0.00535593247616 -1.55808375768
- added joint to_tag_00003: type fixed, parent base_link, child tag36_11_00003, origin xyz=0.0283197929361 0.0413445222178 0.3631483889 rpy=1.54990976662 0.0425628936301 -1.55885953647
- added joint to_tag_00004: type fixed, parent base_link, child tag36_11_00004, origin xyz=0.0336553992455 0.0938285560341 0.651020939576 rpy=1.54988527951 0.0635826585718 -1.55930058089
- joint to_hole_01: origin xyz=-0.0231859078401 -0.0282814474512 0.441118345594 rpy=-0.06403080615 -0.0647848229269 1.55908144855 -> xyz=-0.128572904201 -0.0436470375775 0.696976386728 rpy=-0.0640321358084 -0.0647859936191 1.55908414531
- joint to_hole_02: origin xyz=-0.000463757557886 -0.0305306738819 0.471682850952 rpy=-0.06403080615 -0.0647848229269 1.55908144855 -> xyz=-0.0905311522137 -0.0445775004336 0.704449896867 rpy=-0.0640321358084 -0.0647859936191 1.55908414531
- joint to_hole_03: origin xyz=0.0461839113985 -0.0310339220481 0.471016257947 rpy=-0.06403080615 -0.0647848229269 1.55908144855 -> xyz=-0.0518540837269 -0.0455506243085 0.712466240932 rpy=-0.0640321358084 -0.0647859936191 1.55908414531
- joint to_hole_04: origin xyz=0.0685148465977 -0.0290956950629 0.437109953868 rpy=-0.06403080615 -0.0647848229269 1.55908144855 -> xyz=-0.0156843072925 -0.0449168542623 0.696168518198 rpy=-0.0640321358084 -0.0647859936191 1.55908414531
- joint to_hole_05: origin xyz=0.0445673657398 -0.0269147516117 0.407819156194 rpy=-0.06403080615 -0.0647848229269 1.55908144855 -> xyz=0.073132285793 -0.0457348312841 0.692742156209 rpy=-0.0640321358084 -0.0647859936191 1.55908414531
- joint to_hole_06: origin xyz=-0.000455903779824 -0.0264076500538 0.408133038324 rpy=-0.06403080615 -0.0647848229269 1.55908144855 -> xyz=0.110771926127 -0.0467343114 0.701352005354 rpy=-0.0640321358084 -0.0647859936191 1.55908414531
- joint to_hole_07: origin xyz=-0.0208802619903 -0.0238630597283 0.37260115984 rpy=-0.06403080615 -0.0647848229269 1.55908144855 -> xyz=0.148020448557 -0.0464511320252 0.690263117145 rpy=-0.0640321358084 -0.0647859936191 1.55908414531
- joint to_hole_08: origin xyz=-0.00240257087843 -0.0215015648055 0.332866785156 rpy=-0.06403080615 -0.0647848229269 1.55908144855 -> xyz=0.184546250628 -0.0461781422546 0.679461748475 rpy=-0.0640321358084 -0.0647859936191 1.55908414531
- joint to_hole_09: origin xyz=0.0441438434551 -0.0220229148067 0.332497480315 rpy=-0.06403080615 -0.0647848229269 1.55908144855 -> xyz=-0.0175903946768 -0.0419381068152 0.650601846788 rpy=-0.0640321358084 -0.0647859936191 1.55908414531
- joint to_hole_10: origin xyz=0.0643483206286 -0.0247997737006 0.37164903109 rpy=-0.06403080615 -0.0647848229269 1.55908144855 -> xyz=-0.0186770505831 -0.0386469190131 0.600071673734 rpy=-0.0640321358084 -0.0647859936191 1.55908414531
- joint to_hole_11: origin xyz=-0.0183193680998 -0.0342875833339 0.532812497719 rpy=-0.06403080615 -0.0647848229269 1.55908144855 -> xyz=-0.0206500891437 -0.034355860106 0.534290725435 rpy=-0.0640321358084 -0.0647859936191 1.55908414531
- joint to_hole_12: origin xyz=0.0691214440517 -0.035208122937 0.53121160951 rpy=-0.06403080615 -0.0647848229269 1.55908144855 -> xyz=0.0684187219756 -0.0352716130705 0.53232583042 rpy=-0.0640321358084 -0.0647859936191 1.55908414531
- joint to_hole_13: origin xyz=-0.0173508237974 -0.0384699820474 0.597101150222 rpy=-0.06403080615 -0.0647848229269 1.55908144855 -> xyz=0.0699119300083 -0.0395033625965 0.597279278123 rpy=-0.0640321358084 -0.0647859936191 1.55908414531
- joint to_hole_14: origin xyz=-0.0165201674869 -0.0417052933682 0.646817190801 rpy=-0.06403080615 -0.0647848229269 1.55908144855 -> xyz=0.0711921466145 -0.0426783998721 0.645984306425 rpy=-0.0640321358084 -0.0647859936191 1.55908414531
- joint to_hole_15: origin xyz=-0.0157844883883 -0.0445989234655 0.691284029836 rpy=-0.06403080615 -0.0647848229269 1.55908144855 -> xyz=0.00204170458296 -0.0305479779874 0.471504242059 rpy=-0.0640321358084 -0.0647859936191 1.55908414531
- joint to_hole_16: origin xyz=0.0717634019701 -0.0454885386124 0.689187166127 rpy=-0.06403080615 -0.0647848229269 1.55908144855 -> xyz=-0.0207547067117 -0.0282556146689 0.440287891815 rpy=-0.0640321358084 -0.0647859936191 1.55908414531
- joint to_hole_17: origin xyz=0.0710534490762 -0.0426129907748 0.644994384573 rpy=-0.06403080615 -0.0647848229269 1.55908144855 -> xyz=-0.000420678146768 -0.0263864734588 0.407808425541 rpy=-0.0640321358084 -0.0647859936191 1.55908414531
- joint to_hole_18: origin xyz=0.0699350800666 -0.039412993952 0.595874600682 rpy=-0.06403080615 -0.0647848229269 1.55908144855 -> xyz=0.0454341550422 -0.0268354392926 0.406450269354 rpy=-0.0640321358084 -0.0647859936191 1.55908414531
- joint to_tag_00001: origin xyz=0.160353229673 -0.0402800139396 0.592911176226 rpy=1.63558131631 -0.00225646482702 -0.0118612667906 -> xyz=0.160903806119 -0.0403379930677 0.593717015226 rpy=1.63558262861 0.003492408233 -0.0114843581192
- joint to_tag_00006: origin xyz=0.289039801823 -0.0185894364178 0.235356143456 rpy=-2.88571492705 -1.5038280042 -1.83893893187 -> xyz=0.20594122137 -0.019883196378 0.270321366366 rpy=1.63559918028 -0.0219444636234 -0.0131355670517
- joint to_tag_00100: origin xyz=0.0208917170125 -0.0327790965142 0.440695684094 rpy=1.63559977055 0.0239548219158 -0.0101604937887 -> xyz=0.019355154887 -0.0352760613687 0.441859304771 rpy=1.66566275142 -0.00873291430813 0.0154183638448
- joint to_tag_00101: origin xyz=0.0295741667779 -0.0501954344754 0.707566863227 rpy=1.6355812991 -0.00213025081185 -0.0118530770043 -> xyz=0.0305993768382 -0.0495634897303 0.708105635544 rpy=1.60377606889 0.0126223907212 -0.00366126631718

Commit message: change tag 230 add demo files for intel realsense

File: urdf/P72-with-table.urdf (robot description, URDF)
Before this commit: robot p72, 48 links, 47 joints
Links:
- added link hole_38_link; visual sphere radius=0.005
- added link tag36_11_00013; visual mesh filename=package://gerard_bauzil/meshes/apriltag_36h11/tag36_11_0001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 scale=0.0845 0.0845 1.
Joints:
- added joint to_hole_38: type fixed, parent base_link, child hole_38_link, origin xyz=0.125500811172 0.34818077695 0.247162534997 rpy=1.67565101358 0.0289015115821 -3.03492955206
- added joint to_tag_00013: type fixed, parent base_link, child tag36_11_00013, origin xyz=-0.156582180737 -0.0166076277492 0.285280251246 rpy=-3.09680119279 1.5059440078 1.60396905162
- joint to_hole_00: origin xyz=-0.166815918156 -0.0427314643607 0.689768700188 rpy=-0.0640321358084 -0.0647859936191 1.55908414531 -> xyz=-0.155770641124 -0.0424771571746 0.683856170357 rpy=-0.0640318226797 -0.0647857915715 1.55908237278
- joint to_hole_01: origin xyz=-0.128572904201 -0.0436470375775 0.696976386728 rpy=-0.0640321358084 -0.0647859936191 1.55908414531 -> xyz=-0.119194759843 -0.0434301076044 0.691939929207 rpy=-0.0640318226797 -0.0647857915715 1.55908237278
- joint to_hole_02: origin xyz=-0.0905311522137 -0.0445775004336 0.704449896867 rpy=-0.0640321358084 -0.0647859936191 1.55908414531 -> xyz=-0.0827760353141 -0.044394244251 0.700224474437 rpy=-0.0640318226797 -0.0647857915715 1.55908237278
- joint to_hole_03: origin xyz=-0.0518540837269 -0.0455506243085 0.712466240932 rpy=-0.0640321358084 -0.0647859936191 1.55908414531 -> xyz=-0.0447587609109 -0.045361869915 0.708274171702 rpy=-0.0640318226797 -0.0647857915715 1.55908237278
- joint to_hole_04: origin xyz=-0.0156843072925 -0.0449168542623 0.696168518198 rpy=-0.0640321358084 -0.0647859936191 1.55908414531 -> xyz=-0.00929615138765 -0.0448202747823 0.69352376718 rpy=-0.0640318226797 -0.0647857915715 1.55908237278
- joint to_hole_05: origin xyz=0.073132285793 -0.0457348312841 0.692742156209 rpy=-0.0640321358084 -0.0647859936191 1.55908414531 -> xyz=0.0778339430528 -0.0458425972294 0.69354901095 rpy=-0.0640318226797 -0.0647857915715 1.55908237278
- joint to_hole_06: origin xyz=0.110771926127 -0.0467343114 0.701352005354 rpy=-0.0640321358084 -0.0647859936191 1.55908414531 -> xyz=0.115157469878 -0.0468563840923 0.702435441138 rpy=-0.0640318226797 -0.0647857915715 1.55908237278
- joint to_hole_07: origin xyz=0.148020448557 -0.0464511320252 0.690263117145 rpy=-0.0640321358084 -0.0647859936191 1.55908414531 -> xyz=0.158061748089 -0.0468455903653 0.694522567088 rpy=-0.0640318226797 -0.0647857915715 1.55908237278
- joint to_hole_08: origin xyz=0.184546250628 -0.0461781422546 0.679461748475 rpy=-0.0640321358084 -0.0647859936191 1.55908414531 -> xyz=0.194298536815 -0.0463371141941 0.680142838638 rpy=-0.0640318226797 -0.0647857915715 1.55908237278
- joint to_hole_09: origin xyz=-0.0175903946768 -0.0419381068152 0.650601846788 rpy=-0.0640321358084 -0.0647859936191 1.55908414531 -> xyz=-0.0112678649873 -0.0420553293893 0.651264148847 rpy=-0.0640318226797 -0.0647857915715 1.55908237278
- joint to_hole_10: origin xyz=-0.0186770505831 -0.0386469190131 0.600071673734 rpy=-0.0640321358084 -0.0647859936191 1.55908414531 -> xyz=-0.0121904753945 -0.0388417283305 0.601900060387 rpy=-0.0640318226797 -0.0647857915715 1.55908237278
- joint to_hole_11: origin xyz=-0.0206500891437 -0.034355860106 0.534290725435 rpy=-0.0640321358084 -0.0647859936191 1.55908414531 -> xyz=-0.013035913003 -0.0345847104948 0.536440038537 rpy=-0.0640318226797 -0.0647857915715 1.55908237278
- joint to_hole_12: origin xyz=0.0684187219756 -0.0352716130705 0.53232583042 rpy=-0.0640321358084 -0.0647859936191 1.55908414531 -> xyz=0.0742530225476 -0.0354907632702 0.534644558974 rpy=-0.0640318226797 -0.0647857915715 1.55908237278
- joint to_hole_13: origin xyz=0.0699119300083 -0.0395033625965 0.597279278123 rpy=-0.0640321358084 -0.0647859936191 1.55908414531 -> xyz=0.0757637160624 -0.0397228658765 0.599600452569 rpy=-0.0640318226797 -0.0647857915715 1.55908237278
- joint to_hole_14: origin xyz=0.0711921466145 -0.0426783998721 0.645984306425 rpy=-0.0640321358084 -0.0647859936191 1.55908414531 -> xyz=0.0768435596969 -0.0429395890849 0.648984273182 rpy=-0.0640318226797 -0.0647857915715 1.55908237278
- joint to_hole_15: origin xyz=0.00204170458296 -0.0305479779874 0.471504242059 rpy=-0.0640321358084 -0.0647859936191 1.55908414531 -> xyz=0.0052303051493 -0.0307609328316 0.474206797449 rpy=-0.0640318226797 -0.0647857915715 1.55908237278
- joint to_hole_16: origin xyz=-0.0207547067117 -0.0282556146689 0.440287891815 rpy=-0.0640321358084 -0.0647859936191 1.55908414531 -> xyz=-0.0176592831287 -0.0285031741024 0.443541150984 rpy=-0.0640318226797 -0.0647857915715 1.55908237278
- joint to_hole_17: origin xyz=-0.000420678146768 -0.0263864734588 0.407808425541 rpy=-0.0640321358084 -0.0647859936191 1.55908414531 -> xyz=0.0044037638324 -0.0266528097351 0.411038252283 rpy=-0.0640318226797 -0.0647857915715 1.55908237278
- joint to_hole_18: origin xyz=0.0454341550422 -0.0268354392926 0.406450269354 rpy=-0.0640321358084 -0.0647859936191 1.55908414531 -> xyz=0.0512605036466 -0.0270780033035 0.409131543587 rpy=-0.0640318226797 -0.0647857915715 1.55908237278
- joint to_hole_19: origin xyz=0.0676823414569 -0.0291717367669 0.438442735487 rpy=-0.0640321358084 -0.0647859936191 1.55908414531 -> xyz=0.0739601944277 -0.029369781395 0.440355811145 rpy=-0.0640318226797 -0.0647857915715 1.55908237278
- joint to_hole_20: origin xyz=0.0466270535706 -0.0309939122152 0.470328534663 rpy=-0.0640321358084 -0.0647859936191 1.55908414531 -> xyz=0.0527292674577 -0.0311960427404 0.472336972128 rpy=-0.0640318226797 -0.0647857915715 1.55908237278
- joint to_hole_21: origin xyz=-0.0211758097543 -0.0238817962681 0.372951226012 rpy=-0.0640321358084 -0.0647859936191 1.55908414531 -> xyz=-0.0159863970996 -0.0240253262587 0.37422282316 rpy=-0.0640318226797 -0.0647857915715 1.55908237278
- joint to_hole_22: origin xyz=-0.00265232492397 -0.0214048675679 0.331430916265 rpy=-0.0640321358084 -0.0647859936191 1.55908414531 -> xyz=0.00112257660907 -0.0215245367479 0.332589510569 rpy=-0.0640318226797 -0.0647857915715 1.55908237278
- joint to_hole_23: origin xyz=0.0445434344292 -0.021991831719 0.331957625953 rpy=-0.0640321358084 -0.0647859936191 1.55908414531 -> xyz=0.0492759855859 -0.0221065103501 0.332865107013 rpy=-0.0640318226797 -0.0647857915715 1.55908237278
- joint to_hole_24: origin xyz=0.0651477595884 -0.0247764180189 0.37115622644 rpy=-0.0640321358084 -0.0647859936191 1.55908414531 -> xyz=0.0702131829896 -0.0249036753566 0.372197038486 rpy=-0.0640318226797 -0.0647857915715 1.55908237278
- joint to_hole_25: origin xyz=-0.064504007426 -0.0159695547558 0.258823459798 rpy=-0.0640321358084 -0.0647859936191 1.55908414531 -> xyz=-0.0570256735366 -0.0166625593218 0.268151568967 rpy=-0.0640318226797 -0.0647857915715 1.55908237278
- joint to_hole_26: origin xyz=-0.0984845919704 -0.0121441264254 0.205997349468 rpy=-0.0640321358084 -0.0647859936191 1.55908414531 -> xyz=-0.0918515448753 -0.01273064925 0.213837657992 rpy=-0.0640318226797 -0.0647857915715 1.55908237278
- joint to_hole_27: origin xyz=0.102726204679 -0.0174611899519 0.251624383672 rpy=-0.0640321358084 -0.0647859936191 1.55908414531 -> xyz=0.141074624035 -0.0150914142326 0.208168108264 rpy=-0.0640318226797 -0.0647857915715 1.55908237278
- joint to_hole_28: origin xyz=0.104743399249 0.0130284323996 0.241182377786 rpy=-1.70979382248 -0.76557361026 -3.04842222337 -> xyz=0.106753437325 -0.0118388409354 0.256654473283 rpy=1.02387929648 -0.0175241984904 -0.211638133281
- joint to_hole_29: origin xyz=0.0479809773644 0.278664639966 0.455172061897 rpy=-1.43338884326 0.276368114583 1.58182234414 -> xyz=-0.00102212774089 0.299171906655 0.445735350015 rpy=1.64999112253 -0.047274801489 -1.46662948702
- joint to_hole_30: origin xyz=-0.0114167174748 0.281745848087 0.498838668863 rpy=-1.8917737621 0.250659632952 1.50033157495 -> xyz=-0.0101795664808 0.301414946868 0.488873537139 rpy=1.6491249147 0.0050846080814 -1.44111848342
- joint to_hole_31: origin xyz=-0.0312547275123 0.284154076218 0.539726344304 rpy=-2.21546992664 0.534043741073 1.20554044441 -> xyz=-0.0144997110839 0.301836532246 0.533678698395 rpy=2.16408375452 -0.111223794402 -1.53720683256
- joint to_hole_32: origin xyz=-0.0488979605901 0.287087954303 0.581292765755 rpy=-2.25648458741 0.360820672617 1.29857569528 -> xyz=0.0614741373359 0.309365891905 0.58260602093 rpy=1.83790754352 -0.0628918456327 -1.45084638209
- joint to_hole_33: origin xyz=-0.0645676676101 0.288844357991 0.625612000194 rpy=-3.12218734873 -1.20487785721 3.04938840946 -> xyz=0.0657683245849 0.312086259678 0.627754500815 rpy=2.05523922677 -0.00605405127109 -1.5404014809
- joint to_hole_34: origin xyz=-0.086235960475 0.291866090557 0.665538827329 rpy=3.07565034697 -1.24476911814 3.09128169578 -> xyz=-0.0553205449752 0.308308202778 0.657524847262 rpy=2.46622666149 -0.0507037093904 -1.39838873615
- joint to_hole_35: origin xyz=-0.0181148648809 0.292225548538 0.238329406869 rpy=-1.90145827427 -1.49236800609 0.374570802956 -> xyz=-0.0516551023779 0.348024306204 0.24965343331 rpy=1.59449006759 -0.0425150408999 -3.04640899492
- joint to_hole_36: origin xyz=-0.0577110509484 0.289545685621 0.180503344604 rpy=-2.31264009349 -1.54712996346 0.765146825955 -> xyz=-0.0908704512969 0.344537492662 0.196739871502 rpy=1.67661337086 0.00466998860062 -3.03544809595
- joint to_hole_37: origin xyz=-0.0652507273193 0.279317534307 0.0871087391981 rpy=2.64379590214 -1.4845807824 2.08337128465 -> xyz=-0.0870034310336 0.342045947228 0.14045485912 rpy=1.59110441581 -0.105729647242 -3.05176919967
- joint to_tag_00001: origin xyz=0.160903806119 -0.0403379930677 0.593717015226 rpy=1.63558262861 0.003492408233 -0.0114843581192 -> xyz=0.165575347947 -0.0403532460388 0.593100608649 rpy=1.63558125242 -2.08388275409e-05 -0.0117152118689
- joint to_tag_00002: origin xyz=0.0252040551767 0.290936526509 0.367238386507 rpy=1.54992774545 0.00535593247616 -1.55808375768 -> xyz=0.03254163058 0.31128598997 0.358188437175 rpy=1.51955309441 0.00962846587559 -1.51067110245
- joint to_tag_00003: origin xyz=0.0283197929361 0.0413445222178 0.3631483889 rpy=1.54990976662 0.0425628936301 -1.55885953647 -> xyz=0.047577477726 0.0602993078014 0.354346676841 rpy=1.51951986751 0.0371976888809 -1.51208613621
- joint to_tag_00004: origin xyz=0.0336553992455 0.0938285560341 0.651020939576 rpy=1.54988527951 0.0635826585718 -1.55930058089 -> xyz=0.0591518488962 0.114657635633 0.643827371012 rpy=1.51947935317 0.0543679057873 -1.51296798709
- joint to_tag_00006: origin xyz=0.20594122137 -0.019883196378 0.270321366366 rpy=1.63559918028 -0.0219444636234 -0.0131355670517 -> xyz=0.209757497083 -0.0192690851296 0.260156891357 rpy=1.63558183905 -0.000709491591922 -0.011760293272
- joint to_tag_00100: origin xyz=0.019355154887 -0.0352760613687 0.441859304771 rpy=1.66566275142 -0.00873291430813 0.0154183638448 -> xyz=0.0215301612557 -0.0294468599394 0.437656603341 rpy=1.62189609974 -0.0169612044137 0.0202079512408
- joint to_tag_00101: origin xyz=0.0305993768382 -0.0495634897303 0.708105635544 rpy=1.60377606889 0.0126223907212 -0.00366126631718 -> xyz=0.0336208898396 -0.0454417531079 0.709334144842 rpy=1.60780446811 0.0107058958873 -0.0122439922137

File: urdf/driller_with_qr_drill.urdf (robot description, URDF)
Before this commit: robot driller, 7 links, 6 joints
Links:
- link tag36_11_00230: geometry visual mesh filename=package://gerard_bauzil/meshes/apriltag_36h11/tag36_11_0023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 scale=0.05 0.05 1.
Joints:
- joint tag_joint: origin xyz=0 0 0.002 -> xyz=0 0.009 0.002
- joint tag_joint_back: origin xyz=0 0 0.002 -> xyz=0 -0.005 0.002
- joint tag_support_joint: origin xyz=-0.06 0.00 -0.105 rpy=3.141592653589793 0 -1.57079632679 -> xyz=-0.052 0.00 -0.100 rpy=3.141592653589793 0 -1.57079632679
