Commit message: - add and link realsense to tiago - optimize the p72's holes poses - modified driller's tags - add a hpp file for realsense

File: urdf/P72-with-table.urdf (robot description, URDF)
Before this commit: robot p72, 44 links, 43 joints
Links:
- removed link hole_29_link
Joints:
- removed joint to_hole_29
- joint to_hole_00: origin xyz=-0.176928457126 -0.0426254968751 0.689964585371 rpy=-0.0640310506764 -0.0647850606345 1.55908159829 -> xyz=-0.171321990332 -0.0421616098433 0.68180233862 rpy=-0.0640311055917 -0.0647851134354 1.55908164092
- joint to_hole_01: origin xyz=-0.137661653344 -0.0434392083004 0.695416015586 rpy=-0.0640310506764 -0.0647850606345 1.55908159829 -> xyz=-0.134967027196 -0.0432202069067 0.691553990137 rpy=-0.0640311055917 -0.0647851134354 1.55908164092
- joint to_hole_02: origin xyz=-0.0978615166805 -0.0445778213478 0.70577885156 rpy=-0.0640310506764 -0.0647850606345 1.55908159829 -> xyz=-0.0968187933936 -0.0440970998511 0.6981812339 rpy=-0.0640311055917 -0.0647851134354 1.55908164092
- joint to_hole_03: origin xyz=-0.0600048570023 -0.0455451819336 0.713853102069 rpy=-0.0640310506764 -0.0647850606345 1.55908159829 -> xyz=-0.0583008724167 -0.0450609049794 0.706081300806 rpy=-0.0640311055917 -0.0647851134354 1.55908164092
- joint to_hole_04: origin xyz=-0.0232936406332 -0.0447700767339 0.695277559424 rpy=-0.0640310506764 -0.0647850606345 1.55908159829 -> xyz=-0.0215438601006 -0.0444131762612 0.689460780178 rpy=-0.0640311055917 -0.0647851134354 1.55908164092
- joint to_hole_05: origin xyz=0.0670723685411 -0.045763170374 0.694266959116 rpy=-0.0640310506764 -0.0647850606345 1.55908159829 -> xyz=0.0671349938135 -0.04533841603 0.687709053112 rpy=-0.0640311055917 -0.0647851134354 1.55908164092
- joint to_hole_06: origin xyz=0.105905002358 -0.0468052879326 0.703317209679 rpy=-0.0640310506764 -0.0647850606345 1.55908159829 -> xyz=0.105213015618 -0.0464150832607 0.697428093106 rpy=-0.0640311055917 -0.0647851134354 1.55908164092
- joint to_hole_07: origin xyz=0.142856109914 -0.0465292608176 0.692390640369 rpy=-0.0640310506764 -0.0647850606345 1.55908159829 -> xyz=0.143071851031 -0.0461789550105 0.686952612364 rpy=-0.0640311055917 -0.0647851134354 1.55908164092
- joint to_hole_08: origin xyz=0.181026470749 -0.0462934978701 0.681864505279 rpy=-0.0640310506764 -0.0647850606345 1.55908159829 -> xyz=0.180440114227 -0.0459427351908 0.676564301195 rpy=-0.0640311055917 -0.0647851134354 1.55908164092
- joint to_hole_09: origin xyz=-0.0237518438643 -0.0418160580123 0.649830009357 rpy=-0.0640310506764 -0.0647850606345 1.55908159829 -> xyz=-0.0224890955674 -0.0414695669864 0.64426164932 rpy=-0.0640311055917 -0.0647851134354 1.55908164092
- joint to_hole_10: origin xyz=-0.0249829276586 -0.0384936804986 0.598844502718 rpy=-0.0640310506764 -0.0647850606345 1.55908159829 -> xyz=-0.0241170420771 -0.0382401782744 0.594781078755 rpy=-0.0640311055917 -0.0647851134354 1.55908164092
- joint to_hole_11: origin xyz=-0.0268815925134 -0.0341281796893 0.531901881463 rpy=-0.0640310506764 -0.0647850606345 1.55908159829 -> xyz=-0.0253623970087 -0.0339418135908 0.528755313182 rpy=-0.0640311055917 -0.0647851134354 1.55908164092
- joint to_hole_12: origin xyz=0.0633178886817 -0.0350857870526 0.530374400734 rpy=-0.0640310506764 -0.0647850606345 1.55908159829 -> xyz=0.0638140339585 -0.0348699940821 0.52695906566 rpy=-0.0640311055917 -0.0647851134354 1.55908164092
- joint to_hole_13: origin xyz=0.0640392969511 -0.0393637933404 0.596181043155 rpy=-0.0640310506764 -0.0647850606345 1.55908159829 -> xyz=0.0646747371785 -0.0391049991366 0.592077725384 rpy=-0.0640311055917 -0.0647851134354 1.55908164092
- joint to_hole_14: origin xyz=0.0657666897409 -0.0427871920598 0.648633972298 rpy=-0.0640310506764 -0.0647850606345 1.55908159829 -> xyz=0.0651770872357 -0.0423890219858 0.642603616213 rpy=-0.0640311055917 -0.0647851134354 1.55908164092
- joint to_hole_15: origin xyz=-0.00609446116928 -0.0303256906495 0.469540645645 rpy=-0.0640310506764 -0.0647850606345 1.55908159829 -> xyz=-0.00581565408143 -0.0300868263721 0.465808960919 rpy=-0.0640311055917 -0.0647851134354 1.55908164092
- joint to_hole_16: origin xyz=-0.0292502336407 -0.0280059504154 0.437967669102 rpy=-0.0640310506764 -0.0647850606345 1.55908159829 -> xyz=-0.0287206819784 -0.0277687203336 0.434215906699 rpy=-0.0640311055917 -0.0647851134354 1.55908164092
- joint to_hole_17: origin xyz=-0.00731579572326 -0.026142028329 0.405278397034 rpy=-0.0640310506764 -0.0647850606345 1.55908159829 -> xyz=-0.00681076169956 -0.0259520893171 0.402259999413 rpy=-0.0640311055917 -0.0647851134354 1.55908164092
- joint to_hole_18: origin xyz=0.0401464642266 -0.0266296585833 0.404224106752 rpy=-0.0640310506764 -0.0647850606345 1.55908159829 -> xyz=0.0395908374631 -0.0264151962245 0.401019283039 rpy=-0.0640311055917 -0.0647851134354 1.55908164092
- joint to_hole_19: origin xyz=0.0628637854246 -0.0289390410639 0.435716609241 rpy=-0.0640310506764 -0.0647850606345 1.55908159829 -> xyz=0.0624049149707 -0.0287171565045 0.432379905506 rpy=-0.0640311055917 -0.0647851134354 1.55908164092
- joint to_hole_20: origin xyz=0.0412119961551 -0.0308154818438 0.468547794796 rpy=-0.0640310506764 -0.0647850606345 1.55908159829 -> xyz=0.0411795799397 -0.0305606901784 0.464626849878 rpy=-0.0640311055917 -0.0647851134354 1.55908164092
- joint to_hole_21: origin xyz=-0.0286726948737 -0.0234943628506 0.368326291342 rpy=-0.0640310506764 -0.0647850606345 1.55908159829 -> xyz=-0.027650736389 -0.0233318499444 0.365637288787 rpy=-0.0640311055917 -0.0647851134354 1.55908164092
- joint to_hole_22: origin xyz=-0.00902062419697 -0.0210895886965 0.327712988093 rpy=-0.0640310506764 -0.0647850606345 1.55908159829 -> xyz=-0.00882999697092 -0.0209205690949 0.325073854638 rpy=-0.0640311055917 -0.0647851134354 1.55908164092
- joint to_hole_23: origin xyz=0.0389745252649 -0.0216181776686 0.327193772024 rpy=-0.0640310506764 -0.0647850606345 1.55908159829 -> xyz=0.0385057385935 -0.0214423609369 0.324568974555 rpy=-0.0640311055917 -0.0647851134354 1.55908164092
- joint to_hole_24: origin xyz=0.0596606757314 -0.0244382750723 0.366924686067 rpy=-0.0640310506764 -0.0647850606345 1.55908159829 -> xyz=0.0591660819504 -0.0242572619148 0.364224437202 rpy=-0.0640311055917 -0.0647851134354 1.55908164092
- joint to_hole_25: origin xyz=-0.0723356006168 -0.0152695268592 0.249441000587 rpy=-0.0640310506764 -0.0647850606345 1.55908159829 -> xyz=-0.0722041913402 -0.0151389611034 0.247405270827 rpy=-0.0640311055917 -0.0647851134354 1.55908164092
- joint to_hole_26: origin xyz=-0.109180794342 -0.011189717142 0.193211938038 rpy=-0.0640310506764 -0.0647850606345 1.55908159829 -> xyz=-0.108576452332 -0.0111114957985 0.191897617858 rpy=-0.0640311055917 -0.0647851134354 1.55908164092
- joint to_hole_27: origin xyz=0.131627455845 -0.0140994460697 0.194577477321 rpy=-0.0640310506764 -0.0647850606345 1.55908159829 -> xyz=0.130369519233 -0.0139115318996 0.191908885495 rpy=-0.0640311055917 -0.0647851134354 1.55908164092
- joint to_hole_28: origin xyz=0.0992771197248 -0.0317140358996 0.250164406588 rpy=1.67238186911 0.046367694626 0.0122515208532 -> xyz=0.0972463345939 -0.0276215725564 0.250945171602 rpy=1.65749733575 -0.0230228923082 -0.0118790171612
- joint to_tag_00001: origin xyz=0.18653859187 -0.0196014914218 0.269465194263 rpy=1.63558746674 -0.0144699196329 -0.0126531905553 -> xyz=0.187446082171 -0.0196918851323 0.270695220351 rpy=1.63558832343 -0.0144794549061 -0.0126538620328
- joint to_tag_00002: origin xyz=0.0104561589879 0.288536226701 0.360323280647 rpy=1.50053173786 0.00105371770934 -1.53741961529 -> xyz=0.0175572832871 0.295477342514 0.3578830768 rpy=1.51021243286 -0.000758788717127 -1.53180313163
- joint to_tag_00003: origin xyz=0.0184630884827 0.0420107715974 0.356877816035 rpy=1.5004709021 0.0414307727582 -1.54026319755 -> xyz=0.0270258771322 0.0484033000731 0.355262543794 rpy=1.51017094646 0.0367415970718 -1.53407926645
- joint to_tag_00004: origin xyz=0.0368730299806 0.0943526856921 0.643182175429 rpy=1.50040545392 0.0598893113774 -1.54156559929 -> xyz=0.0422633564625 0.102675094248 0.64111250013 rpy=1.51011312766 0.0572336425954 -1.53532470498
- joint to_tag_00005: origin xyz=-0.135645574854 -0.0157158111433 0.267751334311 rpy=1.63558180009 -0.00482257928219 -0.012027253329 -> xyz=-0.134615156397 -0.0157810400267 0.268570942321 rpy=1.63558216075 -0.00505487204676 -0.0120424020574
- joint to_tag_00006: origin xyz=0.134585443857 -0.0411164973514 0.610456902789 rpy=1.63559209727 0.0180326638639 -0.0105442059083 -> xyz=0.13505343666 -0.0411297358145 0.610576717041 rpy=1.63559091766 0.0168739155875 -0.0106194446955
- joint to_tag_00013: origin xyz=0.304944047226 -0.0287312242645 0.388801820905 rpy=1.6355848352 -0.00977457775816 -0.0123488862354 -> xyz=0.305626995798 -0.0287818764035 0.389459655785 rpy=1.63558754949 -0.013119507191 -0.0125658606706
- joint to_tag_00014: origin xyz=0.296827784967 -0.045124035261 0.642929685157 rpy=1.63558319815 0.00794270375588 -0.0111994215125 -> xyz=0.296861067652 -0.0451246665534 0.64293372232 rpy=1.63558334891 0.00786505678754 -0.0112044889443
- joint to_tag_00100: origin xyz=0.0222953128123 -0.0362667618772 0.555983733047 rpy=1.63558356747 -0.00859777214559 -0.0122723765882 -> xyz=0.0227731313426 -0.0362620079839 0.555824325156 rpy=1.63558590143 -0.0123005948483 -0.0125130784124
- joint to_tag_00101: origin xyz=0.0256081102055 -0.0478418738267 0.733793315777 rpy=1.63558263935 -0.00712741235334 -0.0121767582087 -> xyz=0.0253840100929 -0.0478708964741 0.734281397145 rpy=1.63558300569 -0.00814535064071 -0.0122428747253
- joint to_tag_00102: origin xyz=0.0141243882761 -0.0182143058635 0.279217289181 rpy=1.63558183717 -0.000856455009196 -0.0117701935693 -> xyz=0.0154836510765 -0.0182814625721 0.280007398418 rpy=1.63558236902 -0.000589476469026 -0.011752765053

File: urdf/driller_with_qr_drill.urdf (robot description, URDF)
Before this commit: robot driller, 11 links, 10 joints
Links:
- removed link tag36_11_00231
- removed link tag36_11_00232
- removed link tag_support_link_left
- removed link tag_support_link_top_horizontal
Joints:
- removed joint tag_joint_top_horizontal
- removed joint tag_joint_top_left
- removed joint tag_support_left
- removed joint tag_support_top_horizontal
- joint tag_joint: origin xyz=0 0.009 0.002 -> xyz=0 0.010 0.002 rpy=0 0 0
- joint tag_support_joint: origin xyz=-0.052 0.00 -0.100 rpy=3.141592653589793 0 -1.57079632679 -> xyz=-0.052 0.00 -0.105 rpy=3.141592653589793 0.0 -1.57079632679
- joint tag_support_joint_back: origin xyz=-0.0 0.00 -0.194 rpy=3.141592653589793 0 -1.57079632679 -> xyz=-0.0 0.00 -0.20 rpy=3.141592653589793 0 -1.57079632679

Commit message: Updates for Tiago

File: urdf/P72-with-table.urdf (robot description, URDF)
Before this commit: robot p72, 43 links, 42 joints
Joints:
- joint to_hole_13: origin xyz=0.0646747371785 -0.0391049991366 0.592077725384 rpy=-0.0640311055917 -0.0647851134354 1.55908164092 -> xyz=0.0646747371785 -0.0391049991366 0.582077725384 rpy=-0.0640311055917 -0.0647851134354 1.55908164092
- joint to_hole_14: origin xyz=0.0651770872357 -0.0423890219858 0.642603616213 rpy=-0.0640311055917 -0.0647851134354 1.55908164092 -> xyz=0.0651770872357 -0.0423890219858 0.632603616213 rpy=-0.0640311055917 -0.0647851134354 1.55908164092

File: urdf/driller_with_qr_drill.urdf (robot description, URDF)
Before this commit: robot driller, 7 links, 6 joints
Joints:
- joint tag_joint: origin xyz=0 0.010 0.002 rpy=0 0 0 -> xyz=0.002 0.042 0.002 rpy=0 0 0
- joint tag_joint_back: origin xyz=0 0.0 0.0002 -> xyz=0 -0.00 0.0002
- joint tag_support_joint: origin xyz=-0.052 0.00 -0.105 rpy=3.141592653589793 0.0 -1.57079632679 -> xyz=-0.052 0.00 -0.10 rpy=3.141592653589793 0.0 -1.57079632679
- joint tag_support_joint_back: origin xyz=-0.0 0.00 -0.20 rpy=3.141592653589793 0 -1.57079632679 -> xyz=-0.0 0.00 -0.194 rpy=3.141592653589793 0 -1.57079632679

Commit message: - make p72 part seen with realsense - update readme, config - add rod

File: urdf/P72-with-table.urdf (robot description, URDF)
Before this commit: robot p72, 44 links, 43 joints
Links:
- removed link world
Joints:
- removed joint world_joint

File: urdf/ur.xacro (robot description, xacro)
@@ -174,4 +174,33 @@
      <origin xyz="0.0 0.0 0.0" rpy="0.0 0.0 0.0" />
    </joint>
+   <link name="drill_tip_link">
+   <inertial>
+     <origin xyz="0.0 0.0 0.0" rpy="0 0 0" />
+     <mass value="0.1"/>
+     <inertia ixx="0.001" ixy="0.0" ixz="0.0"
+       iyy="0.001" iyz="0.0"
+       izz="0.001" />
+   </inertial>
+   <visual>
+     <origin xyz="0 0 0" rpy="0 0 0" />
+     <geometry>
+       <mesh filename="package://agimus_demos/meshes/ur10e_drillrod.stl"/>
+     </geometry>
+     <material name="Red">
+       <color rgba="0.9 0.1 0.1 1.0"/>
+     </material>
+   </visual>
+   <collision>
+     <origin xyz="0 0 0" rpy="0 0 0" />
+     <geometry>
+       <mesh filename="package://agimus_demos/meshes/ur10e_drillrod.stl"/>
+     </geometry>
+   </collision>
+  </link>
+  <joint name="drill_tip_joint" type="fixed">
+     <parent link="ur10e_tip_link" />
+     <child link = "drill_tip_link" />
+     <origin xyz="0.0 0.0 0.00" rpy="0.0 0.0 0.0" />
+  </joint>
    <xacro:include filename="$(find realsense2_description)/urdf/_d435.urdf.xacro" />
    <sensor_d435 parent="ur10e_d435_mount_link">

File: urdf/ur10_robot_sim.urdf.xacro (robot description, xacro)
@@ -139,20 +139,27 @@
      <origin xyz="0.0 0.0 0.01" rpy="0.0 0.0 0.0" />
    </joint>
-   <!-- <link name="drill_tip_link">
-    <visual>
-      <origin xyz="0 0 0" rpy="0 0 0" />
-      <geometry>
-        <cylinder radius="0.003" length="0.2"/>
-      </geometry>
-      <material name="black">
-        <color rgba="0 0 0 1"/>
-      </material>
-    </visual>
-    <collision>
-      <origin xyz="0 0 0" rpy="0 0 0"/>
-      <geometry>
-        <cylinder radius="0.003" length="0.2"/>
-      </geometry>
-    </collision>
+   <link name="drill_tip_link">
+   <inertial>
+     <origin xyz="0.0 0.0 0.0" rpy="0 0 0" />
+     <mass value="0.1"/>
+     <inertia ixx="0.001" ixy="0.0" ixz="0.0"
+       iyy="0.001" iyz="0.0"
+       izz="0.001" />
+   </inertial>
+   <visual>
+     <origin xyz="0 0 0" rpy="0 0 0" />
+     <geometry>
+       <mesh filename="package://agimus_demos/meshes/ur10e_drillrod.stl"/>
+     </geometry>
+     <material name="Red">
+       <color rgba="0.9 0.1 0.1 1.0"/>
+     </material>
+   </visual>
+   <collision>
+     <origin xyz="0 0 0" rpy="0 0 0" />
+     <geometry>
+       <mesh filename="package://agimus_demos/meshes/ur10e_drillrod.stl"/>
+     </geometry>
+   </collision>
   </link>
   <joint name="drill_tip_joint" type="fixed">
@@ -160,5 +167,5 @@
      <child link = "drill_tip_link" />
      <origin xyz="0.0 0.0 0.00" rpy="0.0 0.0 0.0" />
-  </joint> -->
+  </joint>
    <xacro:include filename="$(find realsense2_description)/urdf/_d435.urdf.xacro" />
    <sensor_d435 parent="ur10e_d435_mount_link">
