Commit message: [urdf] Add calibration chessboard to april-tag-plank

File: urdf/april-tag-plank.urdf (robot description, URDF)
Before this commit: robot plank-with-april-tags, 3 links, 2 joints
Links:
- link base_link: geometry collision box size=0.02 1.00 1.90; collision box size=0.4 0.05 0.02
Joints:
- joint to_tag_013_base: origin xyz=0 0.045 1.456 rpy=1.5707963267948966 0 1.5707963267948966 -> xyz=0.01 0.045 1.456 rpy=1.5707963267948966 0 1.5707963267948966

Commit message: [urdf] Fix april-tag-plank.urdf

File: urdf/april-tag-plank.urdf (robot description, URDF)
Before this commit: robot plank-with-april-tags, 3 links, 2 joints
Links:
- link base_link: geometry collision box size=0.02 1.00 1.90; collision box size=0.4 0.05 0.02
