Commit message: [ur10/pointing] Move camera on end effector
  move the camera behind and above the tool and align the optical axis with the
  center of the gripper frame.

File: urdf/ur10_robot_sim.urdf.xacro (robot description, xacro)
@@ -11,9 +11,9 @@
     <!-- define global properties -->
     <xacro:property name="M_PI" value="3.1415926535897931" />
-    <xacro:property name="camera_position_x" value="0.0908" />
-    <xacro:property name="camera_position_y" value="0.08" />
-    <xacro:property name="camera_position_z" value="0.0" />
-    <xacro:property name="camera_orientation_r" value="${.5 * M_PI}" />
-    <xacro:property name="camera_orientation_p" value="0.0" />
+    <xacro:property name="camera_position_x" value="-0.12" />
+    <xacro:property name="camera_position_y" value="0.0" />
+    <xacro:property name="camera_position_z" value="-0.2" />
+    <xacro:property name="camera_orientation_r" value="0.0" />
+    <xacro:property name="camera_orientation_p" value="${-0.5*M_PI + 0.38}" />
     <xacro:property name="camera_orientation_y" value="0.0" />
     <link name="support_link">
@@ -103,5 +103,5 @@
      </visual>
    </link>
-   <xacro:orbbec_astra name="xtion" parent="tool"
+   <xacro:orbbec_astra name="xtion" parent="ee"
            camera_model="orbbec-astra'"
            extrinsic_calibration_dir="$(find tiago_description_calibration)/urdf/calibration">
@@ -109,5 +109,5 @@
        rpy="${camera_orientation_r} ${camera_orientation_p}
       ${camera_orientation_y}" />
-     <optical_origin xyz="0 0 0" rpy="${-0.5 * M_PI} 0 ${-.5 * M_PI}"/>
+     <optical_origin xyz="0 0 0" rpy="0 0 0"/>
    </xacro:orbbec_astra>
    <joint name="tool_joint" type="fixed">

Commit message: Add D435 plugin

File: urdf/ur10_robot_sim.urdf.xacro (robot description, xacro)
@@ -41,6 +41,4 @@
       <origin xyz="0.0 0.0 0.0" rpy="0.0 0.0 0.0" />
     </joint>
-    <xacro:include filename="$(find tiago_description)/urdf/sensors/orbbec_astra.urdf.xacro" />
-    <!-- <link name="world" /> -->
     <joint name="robot_joint" type="fixed">
       <parent link="support_link" />
@@ -48,6 +46,6 @@
       <origin xyz="0.0 0.0 0.90" rpy="0.0 0.0 -1.5707963" />
     </joint>
-    <link name="tool_link">
-      <!--collision>
+    <!-- <link name="tool_link">
+      <collision>
         <geometry>
           <box size="0.02 0.05 0.2"/>
@@ -60,7 +58,21 @@
         </geometry>
         <origin rpy="0 0 0" xyz="-0.01 0 0"/>
-      </visual-->
-    </link>
-  <joint name="ee_fixed_joint" type="fixed">
+      </visual>
+    </link -->
+  <!-- <link name="tool_link">
+     <collision>
+       <geometry>
+         <cylinder radius="0.002" length="0.16"/>
+       </geometry>
+       <origin rpy="0 0 0" xyz="0 0 -0.05"/>
+     </collision>
+     <visual>
+       <geometry>
+         <cylinder radius="0.002" length="0.16"/>
+       </geometry>
+       <origin rpy="0 0 0" xyz="0 0 -0.05"/>
+     </visual>
+  </link> -->
+    <joint name="ee_fixed_joint" type="fixed">
      <parent link="wrist_3_link" />
      <child link = "ee_link" />
@@ -68,5 +80,5 @@
    </joint>
    <link name="ee_link">
-     <collision>
+     <!-- <collision>
        <geometry>
          <box size="0.01 0.01 0.01"/>
@@ -79,5 +91,5 @@
        </geometry>
        <origin rpy="0 0 0" xyz="-0.01 0 0"/>
-     </visual>
+     </visual> -->
    </link>
    <link name="ur10e_d435_mount_link">
@@ -169,20 +181,7 @@
   </joint>
    <xacro:include filename="$(find realsense2_description)/urdf/_d435.urdf.xacro" />
-   <sensor_d435 parent="ur10e_d435_mount_link">
+   <sensor_d435 parent="ur10e_d435_mount_link" name="camera">
      <origin xyz="0 0.115 0" rpy="0 -1.0472 -1.57079632679"/>
    </sensor_d435>
-   <!-- <gazebo reference="camera_link">
-     <sensor name="camera" type="camera">
-       ...
-     </sensor>
-   </gazebo> -->
-   <xacro:orbbec_astra name="xtion" parent="ee"
-           camera_model="orbbec-astra'"
-           extrinsic_calibration_dir="$(find tiago_description_calibration)/urdf/calibration">
-     <origin xyz="${camera_position_x} ${camera_position_y} ${camera_position_z}"
-       rpy="${camera_orientation_r} ${camera_orientation_p}
-      ${camera_orientation_y}" />
-     <optical_origin xyz="0 0 0" rpy="0 0 0"/>
-   </xacro:orbbec_astra>
    <joint name="tool_joint" type="fixed">
      <parent link="ee_link"/>

Commit message: Add gazebo colors and node to publish /pose of camera

File: urdf/ur10_robot_sim.urdf.xacro (robot description, xacro)
@@ -180,7 +180,15 @@
      <origin xyz="0.0 0.0 0.00" rpy="0.0 0.0 0.0" />
   </joint>
+   <link name="ref_camera_link">
+   </link>
+    <joint name="ref_camera_joint" type="fixed">
+     <parent link="ur10e_d435_mount_link" />
+     <child link = "ref_camera_link" />
+     <origin xyz="0 0.115 0" rpy="0 -1.0472 -1.57079632679"/>
+   </joint>
    <xacro:include filename="$(find realsense2_description)/urdf/_d435.urdf.xacro" />
-   <xacro:sensor_d435 parent="ur10e_d435_mount_link" name="camera">
-     <origin xyz="0 0.115 0" rpy="0 -1.0472 -1.57079632679"/>
+   <xacro:sensor_d435 parent="ref_camera_link" name="camera">
+     <!-- <origin xyz="0 0.115 0" rpy="0 -1.0472 -1.57079632679"/> -->
+      <origin xyz="0 0 0" rpy="0 0 0"/>
    </xacro:sensor_d435>
    <joint name="tool_joint" type="fixed">

Commit message: [urdf] Remove useless link and joint.

File: urdf/ur10_robot_sim.urdf.xacro (robot description, xacro)
@@ -46,32 +46,4 @@
       <origin xyz="0.0 0.0 0.90" rpy="0.0 0.0 -1.5707963" />
     </joint>
-    <!-- <link name="tool_link">
-      <collision>
-        <geometry>
-          <box size="0.02 0.05 0.2"/>
-        </geometry>
-        <origin rpy="0 0 0" xyz="-0.01 0 0"/>
-      </collision>
-      <visual>
-        <geometry>
-          <box size="0.02 0.05 0.2"/>
-        </geometry>
-        <origin rpy="0 0 0" xyz="-0.01 0 0"/>
-      </visual>
-    </link -->
-  <!-- <link name="tool_link">
-     <collision>
-       <geometry>
-         <cylinder radius="0.002" length="0.16"/>
-       </geometry>
-       <origin rpy="0 0 0" xyz="0 0 -0.05"/>
-     </collision>
-     <visual>
-       <geometry>
-         <cylinder radius="0.002" length="0.16"/>
-       </geometry>
-       <origin rpy="0 0 0" xyz="0 0 -0.05"/>
-     </visual>
-  </link> -->
     <joint name="ee_fixed_joint" type="fixed">
      <parent link="wrist_3_link" />
@@ -192,8 +164,3 @@
       <origin xyz="0 0 0" rpy="0 0 0"/>
    </xacro:sensor_d435>
-   <joint name="tool_joint" type="fixed">
-     <parent link="ee_link"/>
-     <child link="tool_link" />
-     <origin xyz="0.0 0.0 0.0" rpy="0.0 0.0 0.0" />
-   </joint>
 </robot>

Commit message: [ur10/pointing] Run gazebo 30 times slower

File: urdf/ur10_robot_sim.urdf.xacro (robot description, xacro)
@@ -26,5 +26,5 @@
         <origin xyz="-0.4 0 0.45"/>
         <geometry>
-	  <box size="1.0 1.2 0.9"/>
+	        <box size="1.0 1.2 0.9"/>
         </geometry>
       </visual>
@@ -32,5 +32,5 @@
         <origin xyz="-0.4 0 0.45"/>
         <geometry>
-	  <box size="1.0 1.2 0.9"/>
+	        <box size="1.0 1.2 0.9"/>
         </geometry>
       </collision>

Commit message: [ur10/pointing] Add freeflyer joint in FOV model for the plaque

File: urdf/ur10_robot_sim.urdf.xacro (robot description, xacro)
@@ -132,7 +132,7 @@
    </inertial>
    <visual>
-     <origin xyz="0 0 0.09" rpy="0 0 0" />
+     <origin xyz="0 0 0.125" rpy="0 0 0" />
      <geometry>
-       <cylinder radius="0.0015" length="0.18"/> <!-- length="0.25" -->
+       <cylinder radius="0.0015" length="0.25"/>
      </geometry>
      <material name="Pine">
@@ -141,7 +141,7 @@
    </visual>
    <collision>
-     <origin xyz="0 0 0.09" rpy="0 0 0" />
+     <origin xyz="0 0 0.125" rpy="0 0 0" />
      <geometry>
-       <cylinder radius="0.0015" length="0.18"/> <!-- length="0.25" -->
+       <cylinder radius="0.0015" length="0.25"/>
      </geometry>
    </collision>
