Commit message: update the bin_picking demo,which can remove between box and ground

File: urdf/bin-picking-part.urdf (robot description, URDF)
Before this commit: robot bin, 2 links, 1 joints
Links:
- removed link bin_housing_link
- link base_link: mass None -> 1.2; geometry collision mesh filename=package://agimus_demos/meshes/HOUSING-01.stl scale=0.3 0.3 0.3; visual mesh filename=package://agimus_demos/meshes/HOUSING-01.stl scale=0.3 0.3 0.3
Joints:
- removed joint bin_fixed_joint
