Commit message: add realsense d435 camera to robot

File: urdf/ur.xacro (robot description, xacro)
@@ -116,3 +116,32 @@
      <origin xyz="0.0 0.0 0.0" rpy="0.0 0.0 0.0" />
    </joint>
+   <link name="ur10e_d435_mount_link">
+     <inertial>
+       <origin xyz="0.0 0.0 0.0" rpy="0 0 0" />
+       <mass value="0.1"/>
+       <inertia ixx="0.001" ixy="0.0" ixz="0.0"
+         iyy="0.001" iyz="0.0"
+         izz="0.001" />
+     </inertial>
+     <visual>
+       <origin xyz="0 0 0" rpy="0 0 0" />
+       <geometry>
+         <mesh filename="package://agimus_demos/meshes/ur10e_d435_mount.stl"/>
+       </geometry>
+       <material name="Red">
+         <color rgba="0.9 0.1 0.1 1.0"/>
+       </material>
+     </visual>
+     <collision>
+       <origin xyz="0 0 0" rpy="0 0 0" />
+       <geometry>
+         <mesh filename="package://agimus_demos/meshes/ur10e_d435_mount.stl"/>
+       </geometry>
+     </collision>
+   </link>
+   <joint name="ur10e_d435_mount_joint" type="fixed">
+     <parent link="wrist_3_link"/>
+     <child link="ur10e_d435_mount_link" />
+     <origin xyz="0.0 0.0 0.0" rpy="0.0 0.0 0.0" />
+   </joint>
 </robot>

File: urdf/ur10_robot_sim.urdf.xacro (robot description, xacro)
@@ -103,4 +103,42 @@
      </visual>
    </link>
+   <link name="ur10e_d435_mount_link">
+     <inertial>
+       <origin xyz="0.0 0.0 0.0" rpy="0 0 0" />
+       <mass value="0.1"/>
+       <inertia ixx="0.001" ixy="0.0" ixz="0.0"
+         iyy="0.001" iyz="0.0"
+         izz="0.001" />
+     </inertial>
+     <visual>
+       <origin xyz="0 0 0" rpy="0 0 0" />
+       <geometry>
+         <mesh filename="package://agimus_demos/meshes/ur10e_d435_mount.stl"/>
+       </geometry>
+       <material name="Red">
+         <color rgba="0.9 0.1 0.1 1.0"/>
+       </material>
+     </visual>
+     <collision>
+       <origin xyz="0 0 0" rpy="0 0 0" />
+       <geometry>
+         <mesh filename="package://agimus_demos/meshes/ur10e_d435_mount.stl"/>
+       </geometry>
+     </collision>
+   </link>
+   <joint name="ur10e_d435_mount_joint" type="fixed">
+     <parent link="wrist_3_link"/>
+     <child link="ur10e_d435_mount_link" />
+     <origin xyz="0.0 0.0 0.0" rpy="0.0 0.0 3.14159265359" />
+   </joint>
+   <xacro:include filename="$(find realsense2_description)/urdf/_d435.urdf.xacro" />
+   <sensor_d435 parent="ur10e_d435_mount_link">
+     <origin xyz="0 0.115 0" rpy="0 -1.0472 -1.57079632679"/>
+   </sensor_d435>
+   <!-- <gazebo reference="camera_link">
+     <sensor name="camera" type="camera">
+       ...
+     </sensor>
+   </gazebo> -->
    <xacro:orbbec_astra name="xtion" parent="ee"
            camera_model="orbbec-astra'"

Commit message: - add driller tip mount - Realsense in docker

File: urdf/ur.xacro (robot description, xacro)
@@ -143,5 +143,38 @@
      <parent link="wrist_3_link"/>
      <child link="ur10e_d435_mount_link" />
+     <origin xyz="0.0 0.0 0.0" rpy="0.0 0.0 3.14159265359" />
+   </joint>
+   <link name="ur10e_tip_link">
+     <inertial>
+       <origin xyz="0.0 0.0 0.0" rpy="0 0 0" />
+       <mass value="0.1"/>
+       <inertia ixx="0.001" ixy="0.0" ixz="0.0"
+         iyy="0.001" iyz="0.0"
+         izz="0.001" />
+     </inertial>
+     <visual>
+       <origin xyz="0 0 0" rpy="0 0 0" />
+       <geometry>
+         <mesh filename="package://agimus_demos/meshes/ur10e_tip.stl"/>
+       </geometry>
+       <material name="Red">
+         <color rgba="0.9 0.1 0.1 1.0"/>
+       </material>
+     </visual>
+     <collision>
+       <origin xyz="0 0 0" rpy="0 0 0" />
+       <geometry>
+         <mesh filename="package://agimus_demos/meshes/ur10e_tip.stl"/>
+       </geometry>
+     </collision>
+   </link>
+   <joint name="ur10e_tip_joint" type="fixed">
+     <parent link="ur10e_d435_mount_link"/>
+     <child link="ur10e_tip_link" />
      <origin xyz="0.0 0.0 0.0" rpy="0.0 0.0 0.0" />
    </joint>
+   <xacro:include filename="$(find realsense2_description)/urdf/_d435.urdf.xacro" />
+   <sensor_d435 parent="ur10e_d435_mount_link">
+     <origin xyz="0 0.115 0" rpy="0 -1.0472 -1.57079632679"/>
+   </sensor_d435>
 </robot>

File: urdf/ur10_robot_sim.urdf.xacro (robot description, xacro)
@@ -62,27 +62,5 @@
       </visual-->
     </link>
-  <link name="collision_cylinder">
-   <visual>
-     <origin xyz="0 0 0" rpy="0 0 0" />
-     <geometry>
-       <cylinder radius="0.045" length="0.115"/>
-     </geometry>
-     <material name="black">
-       <color rgba="0 0 0 1"/>
-     </material>
-   </visual>
-   <collision>
-     <origin xyz="0 0 0" rpy="0 0 0"/>
-     <geometry>
-       <cylinder radius="0.045" length="0.115"/>
-     </geometry>
-   </collision>
- </link>
- <joint name="collision_cylinder_joint" type="fixed">
-    <parent link="wrist_3_link" />
-    <child link = "collision_cylinder" />
-    <origin xyz="0.0 0.0 0.05" rpy="0.0 0.0 ${pi/2.0}" />
- </joint>
-    <joint name="ee_fixed_joint" type="fixed">
+  <joint name="ee_fixed_joint" type="fixed">
      <parent link="wrist_3_link" />
      <child link = "ee_link" />
@@ -132,4 +110,55 @@
      <origin xyz="0.0 0.0 0.0" rpy="0.0 0.0 3.14159265359" />
    </joint>
+   <link name="ur10e_tip_link">
+     <inertial>
+       <origin xyz="0.0 0.0 0.0" rpy="0 0 0" />
+       <mass value="0.1"/>
+       <inertia ixx="0.001" ixy="0.0" ixz="0.0"
+         iyy="0.001" iyz="0.0"
+         izz="0.001" />
+     </inertial>
+     <visual>
+       <origin xyz="0 0 0" rpy="0 0 0" />
+       <geometry>
+         <mesh filename="package://agimus_demos/meshes/ur10e_tip.stl"/>
+       </geometry>
+       <material name="Red">
+         <color rgba="0.9 0.1 0.1 1.0"/>
+       </material>
+     </visual>
+     <collision>
+       <origin xyz="0 0 0" rpy="0 0 0" />
+       <geometry>
+         <mesh filename="package://agimus_demos/meshes/ur10e_tip.stl"/>
+       </geometry>
+     </collision>
+   </link>
+   <joint name="ur10e_tip_joint" type="fixed">
+     <parent link="ur10e_d435_mount_link"/>
+     <child link="ur10e_tip_link" />
+     <origin xyz="0.0 0.0 0.01" rpy="0.0 0.0 0.0" />
+   </joint>
+   <link name="drill_tip_link">
+    <visual>
+      <origin xyz="0 0 0" rpy="0 0 0" />
+      <geometry>
+        <cylinder radius="0.003" length="0.2"/>
+      </geometry>
+      <material name="black">
+        <color rgba="0 0 0 1"/>
+      </material>
+    </visual>
+    <collision>
+      <origin xyz="0 0 0" rpy="0 0 0"/>
+      <geometry>
+        <cylinder radius="0.003" length="0.2"/>
+      </geometry>
+    </collision>
+  </link>
+  <joint name="drill_tip_joint" type="fixed">
+     <parent link="ur10e_tip_link" />
+     <child link = "drill_tip_link" />
+     <origin xyz="0.0 0.0 0.00" rpy="0.0 0.0 0.0" />
+  </joint>
    <xacro:include filename="$(find realsense2_description)/urdf/_d435.urdf.xacro" />
    <sensor_d435 parent="ur10e_d435_mount_link">

Commit message: [ur10/pointing] Synchronize simulation and robot models.

File: urdf/ur.xacro (robot description, xacro)
@@ -68,6 +68,4 @@
      <origin xyz="0.0 0.0 0.90" rpy="0.0 0.0 -1.5707963" />
    </joint>
-   <link name="tool_link">
-   </link>
    <link name="collision_cylinder">
      <visual>
@@ -98,5 +96,5 @@
    </joint>
    <link name="ee_link">
-     <collision>
+     <!-- <collision>
        <geometry>
          <box size="0.01 0.01 0.01"/>
@@ -109,11 +107,6 @@
        </geometry>
        <origin rpy="0 0 0" xyz="-0.01 0 0"/>
-     </visual>
-   </link>
-   <joint name="tool_joint" type="fixed">
-     <parent link="ee_link"/>
-     <child link="tool_link" />
-     <origin xyz="0.0 0.0 0.0" rpy="0.0 0.0 0.0" />
-   </joint>
+     </visual> -->
+   </link>
    <link name="ur10e_d435_mount_link">
      <inertial>
@@ -203,7 +196,15 @@
      <origin xyz="0.0 0.0 0.00" rpy="0.0 0.0 0.0" />
   </joint>
+   <link name="ref_camera_link">
+   </link>
+    <joint name="ref_camera_joint" type="fixed">
+     <parent link="ur10e_d435_mount_link" />
+     <child link = "ref_camera_link" />
+     <origin xyz="0 0.115 0" rpy="0 -1.0472 -1.57079632679"/>
+   </joint>
    <xacro:include filename="$(find realsense2_description)/urdf/_d435.urdf.xacro" />
-   <sensor_d435 parent="ur10e_d435_mount_link">
-     <origin xyz="0 0.115 0" rpy="0 -1.0472 -1.57079632679"/>
-   </sensor_d435>
+   <xacro:sensor_d435 parent="ref_camera_link" name="camera" use_nominal_extrinsics="true">
+     <!-- <origin xyz="0 0.115 0" rpy="0 -1.0472 -1.57079632679"/> -->
+      <origin xyz="0 0 0" rpy="0 0 0"/>
+   </xacro:sensor_d435>
 </robot>

Commit message: [ur10/pointing] Fix gripper of robot.

File: urdf/ur.xacro (robot description, xacro)
@@ -93,5 +93,5 @@
      <parent link="wrist_3_link" />
      <child link = "ee_link" />
-     <origin xyz="0.0 0.0 0.117" rpy="0.0 0.0 ${pi/2.0}" />
+     <origin xyz="0.0 0.0 0.0" rpy="0.0 0.0 ${pi/2.0}" />
    </joint>
    <link name="ee_link">
@@ -176,16 +176,16 @@
    </inertial>
    <visual>
-     <origin xyz="0 0 0" rpy="0 0 0" />
+     <origin xyz="0 0 0.125" rpy="0 0 0" />
      <geometry>
-       <mesh filename="package://agimus_demos/meshes/ur10e_drillrod.stl"/>
+       <cylinder radius="0.0015" length="0.25"/>
      </geometry>
-     <material name="Red">
-       <color rgba="0.9 0.1 0.1 1.0"/>
+     <material name="Pine">
+       <color rgba="0.8 0.65 0.4 1.0"/>
      </material>
    </visual>
    <collision>
-     <origin xyz="0 0 0" rpy="0 0 0" />
+     <origin xyz="0 0 0.125" rpy="0 0 0" />
      <geometry>
-       <mesh filename="package://agimus_demos/meshes/ur10e_drillrod.stl"/>
+       <cylinder radius="0.0015" length="0.25"/>
      </geometry>
    </collision>

File: urdf/ur10_robot_sim.urdf.xacro (robot description, xacro)
@@ -49,5 +49,5 @@
      <parent link="wrist_3_link" />
      <child link = "ee_link" />
-     <origin xyz="0.0 0.0 0.117" rpy="0.0 0.0 ${pi/2.0}" />
+     <origin xyz="0.0 0.0 0.0" rpy="0.0 0.0 ${pi/2.0}" />
    </joint>
    <link name="ee_link">
@@ -132,16 +132,16 @@
    </inertial>
    <visual>
-     <origin xyz="0 0 0" rpy="0 0 0" />
+     <origin xyz="0 0 0.125" rpy="0 0 0" />
      <geometry>
-       <mesh filename="package://agimus_demos/meshes/ur10e_drillrod.stl"/>
+       <cylinder radius="0.0015" length="0.25"/>
      </geometry>
-     <material name="Red">
-       <color rgba="0.9 0.1 0.1 1.0"/>
+     <material name="Pine">
+       <color rgba="0.8 0.65 0.4 1.0"/>
      </material>
    </visual>
    <collision>
-     <origin xyz="0 0 0" rpy="0 0 0" />
+     <origin xyz="0 0 0.125" rpy="0 0 0" />
      <geometry>
-       <mesh filename="package://agimus_demos/meshes/ur10e_drillrod.stl"/>
+       <cylinder radius="0.0015" length="0.25"/>
      </geometry>
    </collision>

Commit message: [urdf] Update position of camera after calibration on UR10.

File: urdf/ur.xacro (robot description, xacro)
@@ -201,5 +201,6 @@
      <parent link="ur10e_d435_mount_link" />
      <child link = "ref_camera_link" />
-     <origin xyz="0 0.115 0" rpy="0 -1.0472 -1.57079632679"/>
+     <origin xyz="0.00048381  0.11659973 -0.01043009"
+	     rpy="-0.00301722 -1.00532779 -1.56707044"/>
    </joint>
    <xacro:include filename="$(find realsense2_description)/urdf/_d435.urdf.xacro" />

File: urdf/ur10_robot_sim.urdf.xacro (robot description, xacro)
@@ -157,5 +157,6 @@
      <parent link="ur10e_d435_mount_link" />
      <child link = "ref_camera_link" />
-     <origin xyz="0 0.115 0" rpy="0 -1.0472 -1.57079632679"/>
+     <origin xyz="0.00048381  0.11659973 -0.01043009"
+	     rpy="-0.00301722 -1.00532779 -1.56707044"/>
    </joint>
    <xacro:include filename="$(find realsense2_description)/urdf/_d435.urdf.xacro" />

Commit message: [urdf] New position of camera after second calibration.

File: urdf/ur.xacro (robot description, xacro)
@@ -201,6 +201,6 @@
      <parent link="ur10e_d435_mount_link" />
      <child link = "ref_camera_link" />
-     <origin xyz="0.00048381  0.11659973 -0.01043009"
-	     rpy="-0.00301722 -1.00532779 -1.56707044"/>
+     <origin xyz="0.00033351  0.11805402 -0.01064025"
+	     rpy="-0.00127120646 -1.00435876 -1.56137241"/>
    </joint>
    <xacro:include filename="$(find realsense2_description)/urdf/_d435.urdf.xacro" />

File: urdf/ur10_robot_sim.urdf.xacro (robot description, xacro)
@@ -157,6 +157,6 @@
      <parent link="ur10e_d435_mount_link" />
      <child link = "ref_camera_link" />
-     <origin xyz="0.00048381  0.11659973 -0.01043009"
-	     rpy="-0.00301722 -1.00532779 -1.56707044"/>
+     <origin xyz="0.00033351  0.11805402 -0.01064025"
+	     rpy="-0.00127120646 -1.00435876 -1.56137241"/>
    </joint>
    <xacro:include filename="$(find realsense2_description)/urdf/_d435.urdf.xacro" />

Commit message: [ur10/pointing] Set fixed gripper orientation

File: urdf/ur.xacro (robot description, xacro)
@@ -20,4 +20,8 @@
    <xacro:arg name="safety_pos_margin" default="0.15"/>
    <xacro:arg name="safety_k_position" default="20"/>
+   <!-- Offset of the tip link (obtained by calibration) -->
+   <xacro:arg name="tip_offset_x" default="-0.001"/>
+   <xacro:arg name="tip_offset_y" default="0.004"/>
+   <xacro:arg name="tip_offset_z" default="0.241"/>
    <!-- arm -->
    <xacro:ur_robot
@@ -165,5 +169,5 @@
      <parent link="ur10e_d435_mount_link"/>
      <child link="ur10e_tip_link" />
-     <origin xyz="0.0 0.0 0.0" rpy="0.0 0.0 0.0" />
+     <origin xyz="$(arg tip_offset_x) $(arg tip_offset_y) 0.0" rpy="0.0 0.0 0.0" />
    </joint>
    <link name="drill_tip_link">
@@ -176,5 +180,5 @@
    </inertial>
    <visual>
-     <origin xyz="0 0 0.125" rpy="0 0 0" />
+     <origin xyz="0 0 0.113" rpy="0 0 0" />
      <geometry>
        <cylinder radius="0.0015" length="0.25"/>
@@ -185,5 +189,5 @@
    </visual>
    <collision>
-     <origin xyz="0 0 0.125" rpy="0 0 0" />
+     <origin xyz="0 0 0.113" rpy="0 0 0" />
      <geometry>
        <cylinder radius="0.0015" length="0.25"/>
@@ -196,4 +200,11 @@
      <origin xyz="0.0 0.0 0.00" rpy="0.0 0.0 0.0" />
   </joint>
+   <link name="drill_tip_tip_link">
+   </link>
+  <joint name="drill_tip_tip_joint" type="fixed">
+     <parent link="drill_tip_link" />
+     <child link = "drill_tip_tip_link" />
+     <origin xyz="0.0 0.0 $(arg tip_offset_z)" rpy="0.0 0.0 -${pi/2.0}" />
+  </joint>
    <link name="ref_camera_link">
    </link>

File: urdf/ur10_robot_sim.urdf.xacro (robot description, xacro)
@@ -17,4 +17,8 @@
     <xacro:property name="camera_orientation_p" value="${-0.5*M_PI + 0.38}" />
     <xacro:property name="camera_orientation_y" value="0.0" />
+   <!-- Offset of the tip link (obtained by calibration) -->
+   <xacro:arg name="tip_offset_x" default="-0.001"/>
+   <xacro:arg name="tip_offset_y" default="0.004"/>
+   <xacro:arg name="tip_offset_z" default="0.241"/>
     <link name="support_link">
       <inertial>
@@ -121,5 +125,5 @@
      <parent link="ur10e_d435_mount_link"/>
      <child link="ur10e_tip_link" />
-     <origin xyz="0.0 0.0 0.01" rpy="0.0 0.0 0.0" />
+     <origin xyz="$(arg tip_offset_x) $(arg tip_offset_y) 0.0" rpy="0.0 0.0 0.0" />
    </joint>
    <link name="drill_tip_link">
@@ -132,5 +136,5 @@
    </inertial>
    <visual>
-     <origin xyz="0 0 0.125" rpy="0 0 0" />
+     <origin xyz="0 0 0.113" rpy="0 0 0" />
      <geometry>
        <cylinder radius="0.0015" length="0.25"/>
@@ -141,5 +145,5 @@
    </visual>
    <collision>
-     <origin xyz="0 0 0.125" rpy="0 0 0" />
+     <origin xyz="0 0 0.113" rpy="0 0 0" />
      <geometry>
        <cylinder radius="0.0015" length="0.25"/>
@@ -151,4 +155,11 @@
      <child link = "drill_tip_link" />
      <origin xyz="0.0 0.0 0.00" rpy="0.0 0.0 0.0" />
+  </joint>
+   <link name="drill_tip_tip_link">
+   </link>
+  <joint name="drill_tip_tip_joint" type="fixed">
+     <parent link="drill_tip_link" />
+     <child link = "drill_tip_tip_link" />
+     <origin xyz="0.0 0.0 $(arg tip_offset_z)" rpy="0.0 0.0 -${pi/2.0}" />
   </joint>
    <link name="ref_camera_link">

Commit message: [ur10/pointing] Rename robot end-effector frames.
  - ur10e_tip_link -> ur10e_tool_link
  - drill_tip_link ->
  - drill_tip_tip_link -> ur10e_tooltip_link

File: urdf/ur.xacro (robot description, xacro)
@@ -142,5 +142,5 @@
      <origin xyz="0.0 0.0 0.0" rpy="0.0 0.0 3.14159265359" />
    </joint>
-   <link name="ur10e_tip_link">
+   <link name="ur10e_tool_link">
      <inertial>
        <origin xyz="0.0 0.0 0.0" rpy="0 0 0" />
@@ -150,4 +150,5 @@
          izz="0.001" />
      </inertial>
+     <!-- Tool support -->
      <visual>
        <origin xyz="0 0 0" rpy="0 0 0" />
@@ -165,44 +166,31 @@
        </geometry>
      </collision>
-   </link>
-   <joint name="ur10e_tip_joint" type="fixed">
+     <!-- wooden spike -->
+     <visual>
+       <origin xyz="0 0 0.113" rpy="0 0 0" />
+       <geometry>
+	 <cylinder radius="0.0015" length="0.25"/>
+       </geometry>
+       <material name="Pine">
+	 <color rgba="0.8 0.65 0.4 1.0"/>
+       </material>
+     </visual>
+     <collision>
+       <origin xyz="0 0 0.113" rpy="0 0 0" />
+       <geometry>
+	 <cylinder radius="0.0015" length="0.25"/>
+       </geometry>
+     </collision>
+   </link>
+   <joint name="ur10e_tool_joint" type="fixed">
      <parent link="ur10e_d435_mount_link"/>
-     <child link="ur10e_tip_link" />
+     <child link="ur10e_tool_link" />
      <origin xyz="$(arg tip_offset_x) $(arg tip_offset_y) 0.0" rpy="0.0 0.0 0.0" />
    </joint>
-   <link name="drill_tip_link">
-   <inertial>
-     <origin xyz="0.0 0.0 0.0" rpy="0 0 0" />
-     <mass value="0.1"/>
-     <inertia ixx="0.001" ixy="0.0" ixz="0.0"
-       iyy="0.001" iyz="0.0"
-       izz="0.001" />
-   </inertial>
-   <visual>
-     <origin xyz="0 0 0.113" rpy="0 0 0" />
-     <geometry>
-       <cylinder radius="0.0015" length="0.25"/>
-     </geometry>
-     <material name="Pine">
-       <color rgba="0.8 0.65 0.4 1.0"/>
-     </material>
-   </visual>
-   <collision>
-     <origin xyz="0 0 0.113" rpy="0 0 0" />
-     <geometry>
-       <cylinder radius="0.0015" length="0.25"/>
-     </geometry>
-   </collision>
-  </link>
-  <joint name="drill_tip_joint" type="fixed">
-     <parent link="ur10e_tip_link" />
-     <child link = "drill_tip_link" />
-     <origin xyz="0.0 0.0 0.00" rpy="0.0 0.0 0.0" />
-  </joint>
-   <link name="drill_tip_tip_link">
-   </link>
-  <joint name="drill_tip_tip_joint" type="fixed">
-     <parent link="drill_tip_link" />
-     <child link = "drill_tip_tip_link" />
+   <link name="ur10e_tooltip_link">
+   </link>
+  <joint name="ur10e_tooltip_joint" type="fixed">
+     <parent link="ur10e_tool_link" />
+     <child link = "ur10e_tooltip_link" />
      <origin xyz="0.0 0.0 $(arg tip_offset_z)" rpy="0.0 0.0 -${pi/2.0}" />
   </joint>

File: urdf/ur10_robot_sim.urdf.xacro (robot description, xacro)
@@ -98,5 +98,5 @@
      <origin xyz="0.0 0.0 0.0" rpy="0.0 0.0 3.14159265359" />
    </joint>
-   <link name="ur10e_tip_link">
+   <link name="ur10e_tool_link">
      <inertial>
        <origin xyz="0.0 0.0 0.0" rpy="0 0 0" />
@@ -106,4 +106,5 @@
          izz="0.001" />
      </inertial>
+     <!-- Tool support -->
      <visual>
        <origin xyz="0 0 0" rpy="0 0 0" />
@@ -121,44 +122,31 @@
        </geometry>
      </collision>
+     <!-- wooden spike -->
+     <visual>
+       <origin xyz="0 0 0.113" rpy="0 0 0" />
+       <geometry>
+	 <cylinder radius="0.0015" length="0.25"/>
+       </geometry>
+       <material name="Pine">
+	 <color rgba="0.8 0.65 0.4 1.0"/>
+       </material>
+     </visual>
+     <collision>
+       <origin xyz="0 0 0.113" rpy="0 0 0" />
+       <geometry>
+	 <cylinder radius="0.0015" length="0.25"/>
+       </geometry>
+     </collision>
    </link>
-   <joint name="ur10e_tip_joint" type="fixed">
+   <joint name="ur10e_tool_joint" type="fixed">
      <parent link="ur10e_d435_mount_link"/>
-     <child link="ur10e_tip_link" />
+     <child link="ur10e_tool_link" />
      <origin xyz="$(arg tip_offset_x) $(arg tip_offset_y) 0.0" rpy="0.0 0.0 0.0" />
    </joint>
-   <link name="drill_tip_link">
-   <inertial>
-     <origin xyz="0.0 0.0 0.0" rpy="0 0 0" />
-     <mass value="0.1"/>
-     <inertia ixx="0.001" ixy="0.0" ixz="0.0"
-       iyy="0.001" iyz="0.0"
-       izz="0.001" />
-   </inertial>
-   <visual>
-     <origin xyz="0 0 0.113" rpy="0 0 0" />
-     <geometry>
-       <cylinder radius="0.0015" length="0.25"/>
-     </geometry>
-     <material name="Pine">
-       <color rgba="0.8 0.65 0.4 1.0"/>
-     </material>
-   </visual>
-   <collision>
-     <origin xyz="0 0 0.113" rpy="0 0 0" />
-     <geometry>
-       <cylinder radius="0.0015" length="0.25"/>
-     </geometry>
-   </collision>
-  </link>
-  <joint name="drill_tip_joint" type="fixed">
-     <parent link="ur10e_tip_link" />
-     <child link = "drill_tip_link" />
-     <origin xyz="0.0 0.0 0.00" rpy="0.0 0.0 0.0" />
-  </joint>
-   <link name="drill_tip_tip_link">
+   <link name="ur10e_tooltip_link">
    </link>
-  <joint name="drill_tip_tip_joint" type="fixed">
-     <parent link="drill_tip_link" />
-     <child link = "drill_tip_tip_link" />
+  <joint name="ur10e_tooltip_joint" type="fixed">
+     <parent link="ur10e_tool_link" />
+     <child link = "ur10e_tooltip_link" />
      <origin xyz="0.0 0.0 $(arg tip_offset_z)" rpy="0.0 0.0 -${pi/2.0}" />
   </joint>

Commit message: [ur10] Re-orient tooltip_link
  so that it has the same orientation as d435_mount_link.

File: urdf/ur.xacro (robot description, xacro)
@@ -21,7 +21,7 @@
    <xacro:arg name="safety_k_position" default="20"/>
    <!-- Offset of the tip link (obtained by calibration) -->
-   <xacro:arg name="tip_offset_x" default="-0.001"/>
-   <xacro:arg name="tip_offset_y" default="0.004"/>
-   <xacro:arg name="tip_offset_z" default="0.241"/>
+   <xacro:arg name="tip_offset_x" default="0"/>
+   <xacro:arg name="tip_offset_y" default="0"/>
+   <xacro:arg name="tip_offset_z" default="0"/>
    <!-- arm -->
    <xacro:ur_robot
@@ -193,5 +193,5 @@
      <parent link="ur10e_tool_link" />
      <child link = "ur10e_tooltip_link" />
-     <origin xyz="0.0 0.0 $(arg tip_offset_z)" rpy="0.0 0.0 -${pi/2.0}" />
+     <origin xyz="0.0 0.0 ${0.24 + $(arg tip_offset_z)}" rpy="0.0 0.0 0.0" />
   </joint>
    <link name="ref_camera_link">

File: urdf/ur10_robot_sim.urdf.xacro (robot description, xacro)
@@ -18,7 +18,7 @@
     <xacro:property name="camera_orientation_y" value="0.0" />
    <!-- Offset of the tip link (obtained by calibration) -->
-   <xacro:arg name="tip_offset_x" default="-0.001"/>
-   <xacro:arg name="tip_offset_y" default="0.004"/>
-   <xacro:arg name="tip_offset_z" default="0.241"/>
+   <xacro:arg name="tip_offset_x" default="0."/>
+   <xacro:arg name="tip_offset_y" default="0."/>
+   <xacro:arg name="tip_offset_z" default="0."/>
     <link name="support_link">
       <inertial>
@@ -149,5 +149,5 @@
      <parent link="ur10e_tool_link" />
      <child link = "ur10e_tooltip_link" />
-     <origin xyz="0.0 0.0 $(arg tip_offset_z)" rpy="0.0 0.0 -${pi/2.0}" />
+     <origin xyz="0.0 0.0 ${0.24 + $(arg tip_offset_z)}" rpy="0.0 0.0 0.0" />
   </joint>
    <link name="ref_camera_link">
