Commit message: [ur10/pointing] Add wall collision link

File: urdf/ur.xacro (robot description, xacro)
@@ -21,7 +21,7 @@
    <xacro:arg name="safety_k_position" default="20"/>
    <!-- Offset of the tip link (obtained by calibration) -->
-   <xacro:arg name="tip_offset_x" default="0"/>
-   <xacro:arg name="tip_offset_y" default="0"/>
-   <xacro:arg name="tip_offset_z" default="0"/>
+   <xacro:arg name="tip_offset_x" default="0.0008"/>
+   <xacro:arg name="tip_offset_y" default="0.0069"/>
+   <xacro:arg name="tip_offset_z" default="-0.0083"/>
    <!-- arm -->
    <xacro:ur_robot
@@ -43,4 +43,17 @@
    -->
    <link name="world" />
+   <link name="wall_link">
+     <collision>
+       <origin xyz="0 0 1.5"/>
+       <geometry>
+	       <box size="0.1 3 3"/>
+       </geometry>
+     </collision>
+   </link>
+   <joint name="wall_joint" type="fixed">
+     <parent link="world" />
+     <child link = "wall_link" />
+     <origin xyz="-1.4 0.0 0.0" rpy="0.0 0.0 0.0" />
+   </joint>
    <link name="support_link">
      <inertial>
@@ -73,13 +86,4 @@
    </joint>
    <link name="collision_cylinder">
-     <visual>
-       <origin xyz="0 0 0" rpy="0 0 0" />
-       <geometry>
-	 <cylinder radius="0.045" length="0.115"/>
-       </geometry>
-       <material name="black">
-	 <color rgba="0 0 0 1"/>
-       </material>
-     </visual>
      <collision>
        <origin xyz="0 0 0" rpy="0 0 0"/>
@@ -193,5 +197,5 @@
      <parent link="ur10e_tool_link" />
      <child link = "ur10e_tooltip_link" />
-     <origin xyz="0.0 0.0 ${0.24 + $(arg tip_offset_z)}" rpy="0.0 0.0 0.0" />
+     <origin xyz="0.0 0.0 ${0.25 + $(arg tip_offset_z)}" rpy="0.0 0.0 0.0" />
   </joint>
    <link name="ref_camera_link">

File: urdf/ur10_robot_sim.urdf.xacro (robot description, xacro)
@@ -18,7 +18,20 @@
     <xacro:property name="camera_orientation_y" value="0.0" />
    <!-- Offset of the tip link (obtained by calibration) -->
-   <xacro:arg name="tip_offset_x" default="0."/>
-   <xacro:arg name="tip_offset_y" default="0."/>
-   <xacro:arg name="tip_offset_z" default="0."/>
+   <xacro:arg name="tip_offset_x" default="0.0008"/>
+   <xacro:arg name="tip_offset_y" default="0.0069"/>
+   <xacro:arg name="tip_offset_z" default="-0.0083"/>
+   <link name="wall_link">
+     <collision>
+       <origin xyz="0 0 1.5"/>
+       <geometry>
+	       <box size="0.1 3 3"/>
+       </geometry>
+     </collision>
+   </link>
+   <joint name="wall_joint" type="fixed">
+     <parent link="world" />
+     <child link = "wall_link" />
+     <origin xyz="-1.4 0.0 0.0" rpy="0.0 0.0 0.0" />
+   </joint>
     <link name="support_link">
       <inertial>
@@ -149,5 +162,5 @@
      <parent link="ur10e_tool_link" />
      <child link = "ur10e_tooltip_link" />
-     <origin xyz="0.0 0.0 ${0.24 + $(arg tip_offset_z)}" rpy="0.0 0.0 0.0" />
+     <origin xyz="0.0 0.0 ${0.25 + $(arg tip_offset_z)}" rpy="0.0 0.0 0.0" />
   </joint>
    <link name="ref_camera_link">

Commit message: [urdf] Make UR10 support closer to real geometry.
  The previous box was too big. As a result, the initial configuration of the
  robot was closer to the obstacle than the security margin.

File: urdf/ur.xacro (robot description, xacro)
@@ -63,13 +63,25 @@
      </inertial>
      <visual>
-       <origin xyz="-0.4 0 0.45"/>
-       <geometry>
-	 <box size="1.0 1.2 0.9"/>
-       </geometry>
-     </visual>
-     <collision>
-       <origin xyz="-0.4 0 0.45"/>
-       <geometry>
-	 <box size="1.0 1.2 0.9"/>
+       <origin xyz="-0.4 0 0.44"/>
+       <geometry>
+	 <box size="1.0 1.2 0.88"/>
+       </geometry>
+     </visual>
+     <collision>
+       <origin xyz="-0.4 0 0.44"/>
+       <geometry>
+	 <box size="1.0 1.2 0.88"/>
+       </geometry>
+     </collision>
+     <visual>
+       <origin xyz="0 0 0.89"/>
+       <geometry>
+	 <box size="0.15 0.21 0.02"/>
+       </geometry>
+     </visual>
+     <collision>
+       <origin xyz="0 0 0.89"/>
+       <geometry>
+	 <box size="0.15 0.21 0.02"/>
        </geometry>
      </collision>

File: urdf/ur10_robot_sim.urdf.xacro (robot description, xacro)
@@ -41,15 +41,27 @@
       </inertial>
       <visual>
-        <origin xyz="-0.4 0 0.45"/>
+        <origin xyz="-0.4 0 0.44"/>
         <geometry>
-	        <box size="1.0 1.2 0.9"/>
+	        <box size="1.0 1.2 0.88"/>
         </geometry>
       </visual>
       <collision>
-        <origin xyz="-0.4 0 0.45"/>
+        <origin xyz="-0.4 0 0.44"/>
         <geometry>
-	        <box size="1.0 1.2 0.9"/>
+	        <box size="1.0 1.2 0.88"/>
         </geometry>
       </collision>
+     <visual>
+       <origin xyz="0 0 0.89"/>
+       <geometry>
+	 <box size="0.15 0.21 0.02"/>
+       </geometry>
+     </visual>
+     <collision>
+       <origin xyz="0 0 0.89"/>
+       <geometry>
+	 <box size="0.15 0.21 0.02"/>
+       </geometry>
+     </collision>
     </link>
     <joint name="support_joint" type="fixed">
