Commit message: Fix mesh for the plaque

File: urdf/plaque-tubes-with-table.urdf (robot description, URDF)
Before this commit: robot plaque-tubes, 46 links, 45 joints
Links:
- removed link table_link
- added link base_link, mass 2.2; collision box size=.02 .02 .72; collision box size=.02 .02 .72
- link plaque_link: geometry collision mesh filename=package://agimus_demos/meshes/plaque-tubes.stl scale=0.001 0.001 0.001; visual mesh filename=package://agimus_demos/meshes/plaque-tubes.stl scale=0.001 0.001 0.001
Joints:
- joint plaque_joint: parent table_link -> base_link

File: urdf/plaque-tubes.urdf (robot description, URDF)
Before this commit: robot plaque-tubes, 1 links, 0 joints
Links:
- link base_link: geometry collision mesh filename=package://agimus_demos/meshes/plaque-tubes.stl scale=0.001 0.001 0.001; visual mesh filename=package://agimus_demos/meshes/plaque-tubes.stl scale=0.001 0.001 0.001

Commit message: [ur10/pointing] Add plaque as obstacle in fov
And fix margin problem in ur10_fov.py

File: urdf/plaque-tubes-with-table.urdf (robot description, URDF)
Before this commit: robot plaque-tubes, 46 links, 45 joints
Links:
- link plaque_link: geometry collision mesh filename=package://agimus_demos/meshes/plaque-tubes-scaled.stl; visual mesh filename=package://agimus_demos/meshes/plaque-tubes-scaled.stl

File: urdf/ur10_robot_sim.urdf.xacro (robot description, xacro)
@@ -132,7 +132,7 @@
    </inertial>
    <visual>
-     <origin xyz="0 0 0.125" rpy="0 0 0" />
+     <origin xyz="0 0 0.09" rpy="0 0 0" />
      <geometry>
-       <cylinder radius="0.0015" length="0.25"/>
+       <cylinder radius="0.0015" length="0.18"/> <!-- length="0.25" -->
      </geometry>
      <material name="Pine">
@@ -141,7 +141,7 @@
    </visual>
    <collision>
-     <origin xyz="0 0 0.125" rpy="0 0 0" />
+     <origin xyz="0 0 0.09" rpy="0 0 0" />
      <geometry>
-       <cylinder radius="0.0015" length="0.25"/>
+       <cylinder radius="0.0015" length="0.18"/> <!-- length="0.25" -->
      </geometry>
    </collision>

Commit message: [ur10/pointing] Update model part after installation at LAAS.

File: urdf/plaque-tubes-with-table.urdf (robot description, URDF)
Before this commit: robot plaque-tubes, 46 links, 45 joints
Joints:
- joint plaque_joint: origin xyz=-0.5075 0 1.5 rpy=1.5708 0 0 -> xyz=-0.5075 0 1.52 rpy=1.5708 0 0

Commit message: [ur10/pointing] Change numerotation of handle to 2 digits

File: urdf/plaque-tubes-with-table.urdf (robot description, URDF)
Before this commit: robot plaque-tubes, 46 links, 45 joints
Links:
- removed link hole_44_link
- added link hole_00_link; visual sphere radius=0.003
Joints:
- removed joint to_hole_44
- added joint to_hole_00: type fixed, parent plaque_link, child hole_00_link, origin xyz=0.215 -0.2 0 rpy=0 0 0
- joint to_hole_01: origin xyz=0.215 -0.2 0 rpy=0 0 0 -> xyz=0.315 -0.2 0 rpy=0 0 0
- joint to_hole_02: origin xyz=0.315 -0.2 0 rpy=0 0 0 -> xyz=0.415 -0.2 0 rpy=0 0 0
- joint to_hole_03: origin xyz=0.415 -0.2 0 rpy=0 0 0 -> xyz=0.515 -0.2 0 rpy=0 0 0
- joint to_hole_04: origin xyz=0.515 -0.2 0 rpy=0 0 0 -> xyz=0.615 -0.2 0 rpy=0 0 0
- joint to_hole_05: origin xyz=0.615 -0.2 0 rpy=0 0 0 -> xyz=0.715 -0.2 0 rpy=0 0 0
- joint to_hole_06: origin xyz=0.715 -0.2 0 rpy=0 0 0 -> xyz=0.815 -0.2 0 rpy=0 0 0
- joint to_hole_07: origin xyz=0.815 -0.2 0 rpy=0 0 0 -> xyz=0.215 -0.3 0 rpy=0 0 0
- joint to_hole_08: origin xyz=0.215 -0.3 0 rpy=0 0 0 -> xyz=0.315 -0.3 0 rpy=0 0 0
- joint to_hole_09: origin xyz=0.315 -0.3 0 rpy=0 0 0 -> xyz=0.415 -0.3 0 rpy=0 0 0
- joint to_hole_10: origin xyz=0.415 -0.3 0 rpy=0 0 0 -> xyz=0.515 -0.3 0 rpy=0 0 0
- joint to_hole_11: origin xyz=0.515 -0.3 0 rpy=0 0 0 -> xyz=0.615 -0.3 0 rpy=0 0 0
- joint to_hole_12: origin xyz=0.615 -0.3 0 rpy=0 0 0 -> xyz=0.715 -0.3 0 rpy=0 0 0
- joint to_hole_13: origin xyz=0.715 -0.3 0 rpy=0 0 0 -> xyz=0.815 -0.3 0 rpy=0 0 0
- joint to_hole_14: origin xyz=0.815 -0.3 0 rpy=0 0 0 -> xyz=0.215 -0.4 0 rpy=0 0 0
- joint to_hole_15: origin xyz=0.215 -0.4 0 rpy=0 0 0 -> xyz=0.315 -0.4 0 rpy=0 0 0
- joint to_hole_16: origin xyz=0.315 -0.4 0 rpy=0 0 0 -> xyz=0.415 -0.4 0 rpy=0 0 0
- joint to_hole_17: origin xyz=0.415 -0.4 0 rpy=0 0 0 -> xyz=0.515 -0.4 0 rpy=0 0 0
- joint to_hole_18: origin xyz=0.515 -0.4 0 rpy=0 0 0 -> xyz=0.615 -0.4 0 rpy=0 0 0
- joint to_hole_19: origin xyz=0.615 -0.4 0 rpy=0 0 0 -> xyz=0.715 -0.4 0 rpy=0 0 0
- joint to_hole_20: origin xyz=0.715 -0.4 0 rpy=0 0 0 -> xyz=0.815 -0.4 0 rpy=0 0 0
- joint to_hole_21: origin xyz=0.815 -0.4 0 rpy=0 0 0 -> xyz=0.215 -0.5 0 rpy=0 0 0
- joint to_hole_22: origin xyz=0.215 -0.5 0 rpy=0 0 0 -> xyz=0.315 -0.5 0 rpy=0 0 0
- joint to_hole_23: origin xyz=0.315 -0.5 0 rpy=0 0 0 -> xyz=0.415 -0.5 0 rpy=0 0 0
- joint to_hole_24: origin xyz=0.415 -0.5 0 rpy=0 0 0 -> xyz=0.515 -0.5 0 rpy=0 0 0
- joint to_hole_25: origin xyz=0.515 -0.5 0 rpy=0 0 0 -> xyz=0.615 -0.5 0 rpy=0 0 0
- joint to_hole_26: origin xyz=0.615 -0.5 0 rpy=0 0 0 -> xyz=0.715 -0.5 0 rpy=0 0 0
- joint to_hole_27: origin xyz=0.715 -0.5 0 rpy=0 0 0 -> xyz=0.815 -0.5 0 rpy=0 0 0
- joint to_hole_28: origin xyz=0.815 -0.5 0 rpy=0 0 0 -> xyz=0.215 -0.6 0 rpy=0 0 0
- joint to_hole_29: origin xyz=0.215 -0.6 0 rpy=0 0 0 -> xyz=0.315 -0.6 0 rpy=0 0 0
- joint to_hole_30: origin xyz=0.315 -0.6 0 rpy=0 0 0 -> xyz=0.415 -0.6 0 rpy=0 0 0
- joint to_hole_31: origin xyz=0.415 -0.6 0 rpy=0 0 0 -> xyz=0.515 -0.6 0 rpy=0 0 0
- joint to_hole_32: origin xyz=0.515 -0.6 0 rpy=0 0 0 -> xyz=0.615 -0.6 0 rpy=0 0 0
- joint to_hole_33: origin xyz=0.615 -0.6 0 rpy=0 0 0 -> xyz=0.715 -0.6 0 rpy=0 0 0
- joint to_hole_34: origin xyz=0.715 -0.6 0 rpy=0 0 0 -> xyz=0.815 -0.6 0 rpy=0 0 0
- joint to_hole_35: origin xyz=0.815 -0.6 0 rpy=0 0 0 -> xyz=0.025 -0.115 0 rpy=0 0 0
- joint to_hole_36: origin xyz=0.025 -0.115 0 rpy=0 0 0 -> xyz=0.025 -0.686 0 rpy=0 0 0
- joint to_hole_37: origin xyz=0.025 -0.686 0 rpy=0 0 0 -> xyz=0.990 -0.686 0 rpy=0 0 0
- joint to_hole_38: origin xyz=0.990 -0.686 0 rpy=0 0 0 -> xyz=0.990 -0.115 0 rpy=0 0 0
- joint to_hole_39: origin xyz=0.990 -0.115 0 rpy=0 0 0 -> xyz=0.900 -0.025 0 rpy=0 0 0
- joint to_hole_40: origin xyz=0.900 -0.025 0 rpy=0 0 0 -> xyz=0.230 -0.148 0 rpy=0 0 0
- joint to_hole_41: origin xyz=0.230 -0.148 0 rpy=0 0 0 -> xyz=0.445 -0.137 0 rpy=0 0 0
- joint to_hole_42: origin xyz=0.445 -0.137 0 rpy=0 0 0 -> xyz=0.615 -0.267 0 rpy=0 0 0
- joint to_hole_43: origin xyz=0.615 -0.267 0 rpy=0 0 0 -> xyz=0.715 -0.267 0 rpy=0 0 0

Commit message: [ur10/pointing] Reduce table size

File: urdf/plaque-tubes-with-table.urdf (robot description, URDF)
Before this commit: robot plaque-tubes, 46 links, 45 joints
Links:
- link base_link: geometry collision box size=.02 .02 .72; collision box size=.02 .02 .72

Commit message: [ur10/pointing] Add visual bolts for holes 17 and 20

File: urdf/plaque-tubes-with-table.urdf (robot description, URDF)
Before this commit: robot plaque-tubes, 46 links, 45 joints
Links:
- added link bolt_17_link; visual cylinder length=0.004 radius=0.005
- added link bolt_20_link; visual cylinder length=0.004 radius=0.005
Joints:
- added joint to_bolt_17: type fixed, parent plaque_link, child bolt_17_link, origin xyz=0.515 -0.4 0.002 rpy=0 0 0
- added joint to_bolt_20: type fixed, parent plaque_link, child bolt_20_link, origin xyz=0.815 -0.4 0.002 rpy=0 0 0

Commit message: [SNZ demo] Modification to ur10_pointing demo for Saint-Nazaire

File: urdf/plaque-tubes-with-table.urdf (robot description, URDF)
Before this commit: robot plaque-tubes, 48 links, 47 joints
Links:
- link base_link: geometry collision box size=1.995 1 1; visual box size=1.995 1 1
Joints:
- joint plaque_joint: origin xyz=-0.5075 0 1.52 rpy=1.5708 0 0 -> xyz=-0.5 -0.5 1.792 rpy=1.5708 0 0

File: urdf/ur.xacro (robot description, xacro)
@@ -21,7 +21,10 @@
    <xacro:arg name="safety_k_position" default="20"/>
    <!-- Offset of the tip link (obtained by calibration) -->
-   <xacro:arg name="tip_offset_x" default="0.0000"/>
+   <xacro:arg name="tip_offset_x" default="0.0036"/>
+   <xacro:arg name="tip_offset_y" default="0.0090"/>
+   <xacro:arg name="tip_offset_z" default="-0.0068"/>
+     <!-- <xacro:arg name="tip_offset_x" default="0.0000"/>
    <xacro:arg name="tip_offset_y" default="0.0000"/>
-   <xacro:arg name="tip_offset_z" default="0.0000"/>
+   <xacro:arg name="tip_offset_z" default="0.0000"/> -->
    <!-- arm -->
    <xacro:ur_robot
@@ -43,11 +46,25 @@
    -->
    <link name="world" />
-   <link name="wall_link">
-     <collision>
-       <origin xyz="0 0 1.5"/>
-       <geometry>
-	       <box size="0.1 3 3"/>
-       </geometry>
-     </collision>
+      <link name="wall_link">
+   <inertial>
+        <mass value="1000"/>
+        <origin xyz="0 0 0.45"/>
+        <inertia ixx="50"  ixy="0"  ixz="0" iyy="50" iyz="0" izz="50" />
+      </inertial>
+      <visual>
+      <origin xyz="-3 -4.55 3.43" rpy="0 0 1.5708" />
+      <geometry>
+        <mesh filename="package://agimus_demos/meshes/IMC.stl" scale="0.001 0.001 0.001"/>
+      </geometry>
+        <material name="white">
+          <color rgba="1 1 1 1"/>
+        </material>
+    </visual>
+    <collision>
+      <origin xyz="-3 -4.55 3.43" rpy="0 0 1.5708" />
+      <geometry>
+        <mesh filename="package://agimus_demos/meshes/IMC.stl" scale="0.001 0.001 0.001" />
+      </geometry>
+    </collision>
    </link>
    <joint name="wall_joint" type="fixed">
@@ -56,35 +73,35 @@
      <origin xyz="-1.4 0.0 0.0" rpy="0.0 0.0 0.0" />
    </joint>
-   <link name="support_link">
-     <inertial>
-       <mass value="200"/>
-       <origin xyz="0 0 0.45"/>
-       <inertia ixx="50"  ixy="0"  ixz="0" iyy="50" iyz="0" izz="50" />
-     </inertial>
-     <visual>
-       <origin xyz="-0.4 0 0.44"/>
-       <geometry>
-	 <box size="1.0 1.2 0.88"/>
-       </geometry>
-     </visual>
-     <collision>
-       <origin xyz="-0.4 0 0.44"/>
-       <geometry>
-	 <box size="1.0 1.2 0.88"/>
-       </geometry>
-     </collision>
-     <visual>
-       <origin xyz="0 0 0.89"/>
-       <geometry>
-	 <box size="0.15 0.21 0.02"/>
-       </geometry>
-     </visual>
-     <collision>
-       <origin xyz="0 0 0.89"/>
-       <geometry>
-	 <box size="0.15 0.21 0.02"/>
-       </geometry>
-     </collision>
-   </link>
+    <link name="support_link">
+      <inertial>
+        <mass value="200"/>
+        <origin xyz="0 0 0.45"/>
+        <inertia ixx="50"  ixy="0"  ixz="0" iyy="50" iyz="0" izz="50" />
+      </inertial>
+      <visual>
+        <origin xyz="-0.45 0.0 0.44"/>
+        <geometry>
+	        <box size="1.15 0.75 0.855"/>
+        </geometry>
+      </visual>
+      <collision>
+        <origin xyz="-0.45 0.0 0.44"/>
+        <geometry>
+	        <box size="1.15 0.75 0.855"/>
+        </geometry>
+      </collision>
+     <visual>
+       <origin xyz="0 0 0.875"/>
+       <geometry>
+	        <box size="0.15 0.21 0.02"/>
+       </geometry>
+     </visual>
+     <collision>
+       <origin xyz="0 0 0.875"/>
+       <geometry>
+	        <box size="0.15 0.21 0.02"/>
+       </geometry>
+     </collision>
+    </link>
    <joint name="support_joint" type="fixed">
      <parent link="world" />
@@ -95,5 +112,5 @@
      <parent link="support_link" />
      <child link = "base_link" />
-     <origin xyz="0.0 0.0 0.90" rpy="0.0 0.0 -1.5707963" />
+      <origin xyz="0.0 0.0 0.885" rpy="0.0 0.0 -1.5707963" />
    </joint>
    <link name="collision_cylinder">
@@ -217,5 +234,5 @@
      <child link = "ref_camera_link" />
      <origin xyz="0.00033351  0.11805402 -0.01064025"
-	     rpy="-0.00127120646 -1.00435876 -1.56137241"/>
+	     rpy="-0.00127120646 -1.06935876 -1.56137241"/>
    </joint>
    <xacro:include filename="$(find realsense2_description)/urdf/_d435.urdf.xacro" />

File: urdf/ur10_robot_sim.urdf.xacro (robot description, xacro)
@@ -21,11 +21,25 @@
    <xacro:arg name="tip_offset_y" default="0.0069"/>
    <xacro:arg name="tip_offset_z" default="-0.0083"/>
-   <link name="wall_link">
-     <collision>
-       <origin xyz="0 0 1.5"/>
-       <geometry>
-	       <box size="0.1 3 3"/>
-       </geometry>
-     </collision>
+<link name="wall_link">
+   <inertial>
+        <mass value="1000"/>
+        <origin xyz="0 0 0.45"/>
+        <inertia ixx="50"  ixy="0"  ixz="0" iyy="50" iyz="0" izz="50" />
+      </inertial>
+      <visual>
+      <origin xyz="-3 -4.55 3.43" rpy="0 0 1.5708" />
+      <geometry>
+        <mesh filename="package://agimus_demos/meshes/IMC.stl" scale="0.001 0.001 0.001"/>
+      </geometry>
+        <material name="white">
+          <color rgba="1 1 1 1"/>
+        </material>
+    </visual>
+    <collision>
+      <origin xyz="-3 -4.55 3.43" rpy="0 0 1.5708" />
+      <geometry>
+        <mesh filename="package://agimus_demos/meshes/IMC.stl" scale="0.001 0.001 0.001" />
+      </geometry>
+    </collision>
    </link>
    <joint name="wall_joint" type="fixed">
@@ -41,25 +55,25 @@
       </inertial>
       <visual>
-        <origin xyz="-0.4 0 0.44"/>
+        <origin xyz="-0.45 0.0 0.44"/>
         <geometry>
-	        <box size="1.0 1.2 0.88"/>
+	        <box size="1.15 0.75 0.855"/>
         </geometry>
       </visual>
       <collision>
-        <origin xyz="-0.4 0 0.44"/>
+        <origin xyz="-0.45 0.0 0.44"/>
         <geometry>
-	        <box size="1.0 1.2 0.88"/>
+	        <box size="1.15 0.75 0.855"/>
         </geometry>
       </collision>
      <visual>
-       <origin xyz="0 0 0.89"/>
-       <geometry>
-	 <box size="0.15 0.21 0.02"/>
-       </geometry>
-     </visual>
-     <collision>
-       <origin xyz="0 0 0.89"/>
-       <geometry>
-	 <box size="0.15 0.21 0.02"/>
+       <origin xyz="0 0 0.875"/>
+       <geometry>
+	        <box size="0.15 0.21 0.02"/>
+       </geometry>
+     </visual>
+     <collision>
+       <origin xyz="0 0 0.875"/>
+       <geometry>
+	        <box size="0.15 0.21 0.02"/>
        </geometry>
      </collision>
@@ -73,5 +87,5 @@
       <parent link="support_link" />
       <child link = "base_link" />
-      <origin xyz="0.0 0.0 0.90" rpy="0.0 0.0 -1.5707963" />
+      <origin xyz="0.0 0.0 0.885" rpy="0.0 0.0 -1.5707963" />
     </joint>
     <joint name="ee_fixed_joint" type="fixed">
