Commit message: Move part model from top project to this submodule.

File: urdf/robot.urdf.xacro (robot description, xacro)
@@ -48,5 +48,5 @@
   <xacro:property name="camera_pose" value="${load_yaml(camera_pose_file)}"/>
    <link name="world" />
-      <link name="wall_link">
+   <link name="wall_link">
    <inertial>
         <mass value="1000"/>

Commit message: [meshes] move models from agimus-demos.

File: urdf/robot.urdf.xacro (robot description, xacro)
@@ -57,5 +57,5 @@
       <origin xyz="-3 -4.55 3.43" rpy="0 0 1.5708" />
       <geometry>
-        <mesh filename="package://agimus_demos/meshes/IMC.stl" scale="0.001 0.001 0.001"/>
+        <mesh filename="package://agimus_demos/ur10/pointing/meshes/IMC.stl" scale="0.001 0.001 0.001"/>
       </geometry>
         <material name="white">
@@ -66,5 +66,5 @@
       <origin xyz="-3 -4.55 3.43" rpy="0 0 1.5708" />
       <geometry>
-        <mesh filename="package://agimus_demos/meshes/IMC.stl" scale="0.001 0.001 0.001" />
+        <mesh filename="package://agimus_demos/ur10/pointing/meshes/IMC.stl" scale="0.001 0.001 0.001" />
       </geometry>
     </collision>
@@ -159,5 +159,5 @@
        <origin xyz="0 0 0" rpy="0 0 0" />
        <geometry>
-         <mesh filename="package://agimus_demos/meshes/ur10e_d435_mount.stl"/>
+         <mesh filename="package://agimus_demos/ur10/pointing/meshes/ur10e_d435_mount.stl"/>
        </geometry>
        <material name="Red">
@@ -168,5 +168,5 @@
        <origin xyz="0 0 0" rpy="0 0 0" />
        <geometry>
-         <mesh filename="package://agimus_demos/meshes/ur10e_d435_mount.stl"/>
+         <mesh filename="package://agimus_demos/ur10/pointing/meshes/ur10e_d435_mount.stl"/>
        </geometry>
      </collision>
@@ -189,5 +189,5 @@
        <origin xyz="0 0 0" rpy="0 0 0" />
        <geometry>
-         <mesh filename="package://agimus_demos/meshes/ur10e_tip.stl"/>
+         <mesh filename="package://agimus_demos/ur10/pointing/meshes/ur10e_tip.stl"/>
        </geometry>
        <material name="Red">
@@ -198,5 +198,5 @@
        <origin xyz="0 0 0" rpy="0 0 0" />
        <geometry>
-         <mesh filename="package://agimus_demos/meshes/ur10e_tip.stl"/>
+         <mesh filename="package://agimus_demos/ur10/pointing/meshes/ur10e_tip.stl"/>
        </geometry>
      </collision>

Commit message: [urdf] Remove duplicated geometry.

File: urdf/robot.urdf.xacro (robot description, xacro)
@@ -48,31 +48,4 @@
   <xacro:property name="camera_pose" value="${load_yaml(camera_pose_file)}"/>
    <link name="world" />
-   <link name="wall_link">
-   <inertial>
-        <mass value="1000"/>
-        <origin xyz="0 0 0.45"/>
-        <inertia ixx="50"  ixy="0"  ixz="0" iyy="50" iyz="0" izz="50" />
-      </inertial>
-      <visual>
-      <origin xyz="-3 -4.55 3.43" rpy="0 0 1.5708" />
-      <geometry>
-        <mesh filename="package://agimus_demos/ur10/pointing/meshes/IMC.stl" scale="0.001 0.001 0.001"/>
-      </geometry>
-        <material name="white">
-          <color rgba="1 1 1 1"/>
-        </material>
-    </visual>
-    <collision>
-      <origin xyz="-3 -4.55 3.43" rpy="0 0 1.5708" />
-      <geometry>
-        <mesh filename="package://agimus_demos/ur10/pointing/meshes/IMC.stl" scale="0.001 0.001 0.001" />
-      </geometry>
-    </collision>
-   </link>
-   <joint name="wall_joint" type="fixed">
-     <parent link="world" />
-     <child link = "wall_link" />
-     <origin xyz="-1.4 0.0 0.0" rpy="0.0 0.0 0.0" />
-   </joint>
     <link name="support_link">
       <inertial>
