Commit message: [calibration] Collect data in simulation

File: data-simulation/robot.urdf (robot description, URDF)
Before this commit: robot ur10e, 30 links, 29 joints
Links:
- link ur10e_tool_link: geometry collision cylinder length=0.25 radius=0.0015; collision mesh filename=package://agimus_demos/meshes/ur10e_tip.stl

Commit message: [calibration] Collect data in simulation

File: data-simulation/robot.urdf (robot description, URDF)
Before this commit: robot ur10e, 29 links, 28 joints
Links:
- added link collision_cylinder; collision cylinder length=0.115 radius=0.045
- link ur10e_tool_link: geometry collision mesh filename=package://agimus_demos/meshes/ur10e_tip.stl; visual mesh filename=package://agimus_demos/meshes/ur10e_tip.stl
Joints:
- added joint collision_cylinder_joint: type fixed, parent wrist_3_link, child collision_cylinder, origin xyz=0.0 0.0 0.05 rpy=0.0 0.0 1.5707963267948966
- joint ur10e_tool_joint: origin xyz=0.0008 0.0069 0.0 rpy=0.0 0.0 0.0 -> xyz=0.0000 0.0000 0.0 rpy=0.0 0.0 0.0
- joint ur10e_tooltip_joint: origin xyz=0.0 0.0 0.2417 rpy=0.0 0.0 0.0 -> xyz=0.0 0.0 0.25 rpy=0.0 0.0 0.0
